File: Controller/Eagle/Projects/Controller/controller_v1.sch (EAGLE design)
At the start: 47 parts, among them J1 BATT, U1 V_REG_317SMD, U2 ATMEGA128RFA1, U3 RF_AMPLIFIER, Y1 32.768kHz, Y2 16MHz

Commit message: In the controller, adding a partially routed PCB.
Connections:
- net GM_SEL: now also U2.PG0(DIG3); no longer U2.PG2(AMR)
- net PA_EN: now also U2.PG2(AMR); no longer U2.PG0(DIG3)
Changed lines of the file:
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@@
 </segment>
 <segment>
-<wire x1="132.08" y1="17.78" x2="144.78" y2="17.78" width="0.1524" layer="91"/>
-<label x="144.78" y="17.78" size="1.27" layer="95" ratio="5" xref="yes"/>
-<pinref part="U2" gate="G$1" pin="PG0(DIG3)"/>
+<wire x1="132.08" y1="12.7" x2="144.78" y2="12.7" width="0.1524" layer="91"/>
+<label x="144.78" y="12.7" size="1.27" layer="95" ratio="5" xref="yes"/>
+<pinref part="U2" gate="G$1" pin="PG2(AMR)"/>
 </segment>
 </net>
@@
 </segment>
 <segment>
-<wire x1="132.08" y1="12.7" x2="144.78" y2="12.7" width="0.1524" layer="91"/>
-<label x="144.78" y="12.7" size="1.27" layer="95" ratio="5" xref="yes"/>
-<pinref part="U2" gate="G$1" pin="PG2(AMR)"/>
+<pinref part="U2" gate="G$1" pin="PG0(DIG3)"/>
+<wire x1="132.08" y1="17.78" x2="142.24" y2="17.78" width="0.1524" layer="91"/>
+<label x="142.24" y="17.78" size="1.27" layer="95" xref="yes"/>
 </segment>
 </net>

Commit message: Finished first version of of the controller board, all of the way to routing Stil need to pass checks for the schematic, but i will ask about those in class today.
Parts:
- removed JP2: M13X22X13, SparkFun-Connectors:M13X22X13
- removed JP4: AVR_MINI_PROGSMD, Controller:AVR_MINI_PROGSMD
- added J2: AVR_SPI_PRG_6NS, Controller:AVR_SPI_PRG_6NS
- added JP5, JP7: M10", Controller:M10"
- added JP6: (no value), Controller:M081X08
Connections:
- new net PD8: JP7.2
- new net PE6: JP6.3, U2.PE6(T3/INT6)
- new net PE7: JP6.2, U2.PE7(ICP3/INT7/CLKO)
- net 3.3V: now also J2.2, JP6.8, JP7.10; no longer JP2.16, JP4.VCC
- net ADC0: now also JP5.9; no longer JP2.4
- net ADC1: now also JP5.8; no longer JP2.6
- net ADC2: now also JP5.7; no longer JP2.8
- net ADC3: now also JP5.6
- net ADC4: now also JP5.5
- net ADC5: now also JP5.4; no longer JP2.10
- net ADC6: now also JP5.3; no longer JP2.12
- net ADC7: now also JP5.2; no longer JP2.14
- net AREF: now also JP5.10; no longer JP2.2
- net GND: now also J2.6, JP5.1, JP6.1, JP7.1; no longer JP2.18, JP4.GND
- net MISO: now also J2.1; no longer JP4.MISO
- net MOSI: now also J2.4; no longer JP4.MOSI
- net PB4: no longer JP2.20
- net PB5: no longer JP2.22
- net PB6: no longer JP2.24
- net PB7: no longer JP2.26
- net PD0/I2C_SCL: now also JP7.9; no longer JP2.1
- net PD1/I2C_SDA: now also JP7.8; no longer JP2.3
- net PD2/RXD1: now also JP7.7; no longer JP2.5
- net PD3/TXD1: now also JP7.6; no longer JP2.7
- net PD4: now also JP7.5; no longer JP2.9
- net PD5: now also JP7.4; no longer JP2.11
- net PD6: no longer JP2.13
- net PD7: now also JP7.3; no longer JP2.15
- net PE2: now also JP6.7; no longer JP2.19
- net PE3: now also JP6.6; no longer JP2.21
- net PE4: now also JP6.5; no longer JP2.23
- net PE5: now also JP6.4; no longer JP2.25
- net RESET_N: now also J2.5; no longer JP2.17, JP4.RST
- net SCK: now also J2.3; no longer JP4.SCK
