File: Controller/Eagle/Projects/Controller/controller_v6.brd (EAGLE design)
At the start: 250 x 115 mm, 74 parts, among them J2 AVR_SPI_PRG_6NS, J3 GIMBAL_3PIN, J4 GIMBAL_3PIN, J5 GIMBAL_3PIN, J6 GIMBAL_3PIN, U2 ATMEGA128RFA1, Y1 32.768kHz, Y2 16MHz

Commit message: Adding design files for controller v5, and controller v6.
Controller v5 has holes milled in the center of the board (which costs
substantially more). Controller v6 uses the board outline to create these holes
(there are no holes in the middle, just a cut into the board). I've added all of
the design files that I submitted to 4PCB and passed through FREEDFM.

In addition, I've added the CAM file job that I used to create these files. It
generates a GERBER file and EPS file of the board layout. 4PCB wanted the GERBER
File, but I found that the EPS file was easier for me two view. They contain
identical information.
Routing:
- net 3.3V: track 1243.1 -> 1124.9 mm
- net GND: track 1495.4 -> 1396.5 mm
Other:
- outline, holes or cut-outs redrawn
Changed lines of the file:
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@@
 <plain>
 <wire x1="0" y1="0" x2="250" y2="0" width="0" layer="20"/>
-<wire x1="250" y1="0" x2="250" y2="115" width="0" layer="20"/>
+<wire x1="250" y1="0" x2="250" y2="40" width="0" layer="20"/>
+<wire x1="250" y1="75" x2="250" y2="115" width="0" layer="20"/>
 <wire x1="250" y1="115" x2="0" y2="115" width="0" layer="20"/>
-<wire x1="0" y1="115" x2="0" y2="0" width="0" layer="20"/>
+<wire x1="0" y1="115" x2="0" y2="75" width="0" layer="20"/>
 <text x="27.85" y="91" size="1.778" layer="21">PD2</text>
 <text x="28.25" y="22.45" size="1.778" layer="21">PD3</text>
@@
 <dimension x1="0" y1="0" x2="0.85" y2="115" x3="-2.4" y3="57.5" textsize="1.778" layer="20" dtype="vertical" visible="yes"/>
 <dimension x1="0" y1="115" x2="250" y2="115" x3="125" y3="118.45" textsize="1.778" layer="20" dtype="horizontal" visible="yes"/>
+<wire x1="0" y1="40" x2="0" y2="0" width="0" layer="20"/>
+<wire x1="220" y1="33.5" x2="220" y2="81.5" width="0" layer="20" curve="-180" cap="flat"/>
+<wire x1="220" y1="81.5" x2="240" y2="81.5" width="0" layer="20"/>
+<wire x1="240" y1="81.5" x2="240" y2="75" width="0" layer="20"/>
+<wire x1="240" y1="75" x2="250" y2="75" width="0" layer="20"/>
+<wire x1="220" y1="33.5" x2="240" y2="33.5" width="0" layer="20"/>
+<wire x1="240" y1="33.5" x2="240" y2="40" width="0" layer="20"/>
+<wire x1="240" y1="40" x2="250" y2="40" width="0" layer="20"/>
+<wire x1="30" y1="33.5" x2="10" y2="33.5" width="0" layer="20"/>
+<wire x1="10" y1="33.5" x2="10" y2="40" width="0" layer="20"/>
+<wire x1="10" y1="40" x2="0" y2="40" width="0" layer="20"/>
+<wire x1="30" y1="81.5" x2="10" y2="81.5" width="0" layer="20"/>
+<wire x1="10" y1="81.5" x2="10" y2="75" width="0" layer="20"/>
+<wire x1="10" y1="75" x2="0" y2="75" width="0" layer="20"/>
+<wire x1="30" y1="81.5" x2="30" y2="33.5" width="0" layer="20" curve="-180" cap="flat"/>
 </plain>
 <attributes>
@@
 <wire x1="160" y1="110" x2="177.85" y2="110" width="1.016" layer="1"/>
 <wire x1="177.85" y1="110" x2="223.3" y2="110" width="1.016" layer="1"/>
-<wire x1="223.3" y1="110" x2="247" y2="110" width="1.016" layer="1"/>
-<wire x1="247" y1="110" x2="247" y2="3" width="1.016" layer="1"/>
 <wire x1="247" y1="3" x2="226.35" y2="3" width="1.016" layer="1"/>
 <wire x1="226.35" y1="3" x2="181.25" y2="3" width="1.016" layer="1"/>
@@
 <wire x1="111.1" y1="3" x2="82" y2="3" width="1.016" layer="1"/>
 <wire x1="82" y1="3" x2="36" y2="3" width="1.016" layer="1"/>
-<wire x1="36" y1="3" x2="3" y2="3" width="1.016" layer="1"/>
+<wire x1="36" y1="3" x2="3.05" y2="3" width="1.016" layer="1"/>
 <wire x1="3" y1="110" x2="32.7" y2="110" width="1.016" layer="1"/>
 <wire x1="90" y1="95" x2="104.25" y2="95" width="1.016" layer="1"/>
@@
 <wire x1="65.7" y1="69.9" x2="65.7" y2="55" width="1.016" layer="1"/>
 <wire x1="65.7" y1="55" x2="65.7" y2="51.75" width="1.016" layer="1"/>
-<wire x1="86.45" y1="41.25" x2="65.7" y2="41.15" width="1.016" layer="1"/>
+<wire x1="86.45" y1="41.25" x2="72.95320625" y2="41.18495625" width="1.016" layer="1"/>
+<wire x1="72.95320625" y1="41.18495625" x2="65.7" y2="41.15" width="1.016" layer="1"/>
 <wire x1="65.7" y1="41.15" x2="65.7" y2="51.75" width="1.016" layer="1"/>
 <wire x1="65.7" y1="52" x2="65.7" y2="51.75" width="0.254" layer="1"/>
@@
 <wire x1="149.05" y1="65.85" x2="149.05" y2="70.3" width="0.4064" layer="16"/>
 <via x="149.05" y="70.3" extent="1-16" drill="0.6096"/>
-<wire x1="149.05" y1="95" x2="148.55" y2="95" width="0.4064" layer="1"/>
+<wire x1="149.05" y1="95" x2="148.6" y2="95" width="0.4064" layer="1"/>
+<wire x1="148.6" y1="95" x2="148.55" y2="95" width="0.4064" layer="1"/>
 <wire x1="149.05" y1="69.75" x2="149.05" y2="70.3" width="0.254" layer="1"/>
 <wire x1="148.45" y1="69.15" x2="149.05" y2="69.75" width="0.254" layer="1"/>
@@
 <wire x1="130.7" y1="78.75" x2="131.5" y2="77.95" width="0.254" layer="1"/>
 <wire x1="109.7" y1="72.5" x2="109.7" y2="73.73" width="0.254" layer="1"/>
-<wire x1="3" y1="3" x2="3" y2="110" width="1.016" layer="1"/>
+<wire x1="3" y1="3" x2="3.05" y2="3" width="1.016" layer="1"/>
+<wire x1="3.05" y1="3" x2="3.05" y2="32.2" width="1.016" layer="1"/>
+<wire x1="3.05" y1="32.2" x2="72.95320625" y2="32.2" width="1.016" layer="1"/>
+<wire x1="72.95320625" y1="32.2" x2="72.95320625" y2="41.18495625" width="1.016" layer="1"/>
+<wire x1="160" y1="95" x2="148.6" y2="95" width="1.016" layer="1"/>
 </signal>
 <signal name="GND">
@@
 <wire x1="160" y1="90.2" x2="160" y2="110" width="1.016" layer="16"/>
 <wire x1="160" y1="110" x2="227.95" y2="110" width="1.016" layer="16"/>
-<wire x1="227.95" y1="110" x2="247" y2="110" width="1.016" layer="16"/>
-<wire x1="247" y1="110" x2="247" y2="19.4" width="1.016" layer="16"/>
 <wire x1="247" y1="19.4" x2="247" y2="3" width="1.016" layer="16"/>
 <wire x1="247" y1="3" x2="182.65" y2="3" width="1.016" layer="16"/>
@@
 <via x="231.05" y="19.4" extent="1-16" drill="0.6096"/>
 <wire x1="84.2" y1="110" x2="84.2" y2="112" width="1.016" layer="16"/>
-<wire x1="84.2" y1="112" x2="89.95" y2="112" width="1.016" layer="16"/>
-<wire x1="89.95" y1="112" x2="89.95" y2="110" width="1.016" layer="16"/>
+<wire x1="84.2" y1="112" x2="90" y2="112" width="1.016" layer="16"/>
+<wire x1="90" y1="112" x2="90" y2="110" width="1.016" layer="16"/>
 <wire x1="80" y1="101.27" x2="80" y2="101.53" width="1.016" layer="1"/>
 <wire x1="80" y1="101.53" x2="72.05" y2="101.53" width="1.016" layer="1"/>
@@
 <wire x1="130.5" y1="70.1" x2="130.5" y2="70" width="0.254" layer="16"/>
 <via x="130.5" y="70.1" extent="1-16" drill="0.6"/>
-<wire x1="90" y1="111.6" x2="89.95" y2="112" width="0.254" layer="16"/>
+<wire x1="90" y1="111.6" x2="90" y2="112" width="0.254" layer="16"/>
 <wire x1="122" y1="93.1" x2="122" y2="89.3" width="0.254" layer="1"/>
 <wire x1="125.8" y1="97" x2="127.25" y2="97" width="0.254" layer="1"/>
@@
 <wire x1="128.15" y1="96.1" x2="128.15" y2="93.1" width="0.254" layer="1"/>
 <wire x1="128.15" y1="93.1" x2="126.05" y2="91" width="0.254" layer="1"/>
-<wire x1="50.65" y1="90.2" x2="50.605" y2="90.24" width="0" layer="19" extent="16-16"/>
-<wire x1="90" y1="110" x2="89.95" y2="110" width="0" layer="19" extent="16-16"/>
-<wire x1="3" y1="3" x2="3" y2="110" width="1.016" layer="16"/>
+<wire x1="3" y1="3" x2="3" y2="32.15" width="1.016" layer="16"/>
+<wire x1="3" y1="32.15" x2="72.95" y2="32.15" width="1.016" layer="16"/>
+<wire x1="72.95" y1="32.15" x2="72.95" y2="45.2" width="1.016" layer="16"/>
+<wire x1="159.5" y1="89.95" x2="155" y2="89.95" width="1.016" layer="16"/>
+<wire x1="155" y1="89.95" x2="154.5" y2="90" width="1.016" layer="16"/>
+<wire x1="159.5" y1="89.95" x2="160" y2="90" width="1.016" layer="16"/>
+<wire x1="50.65" y1="90.2" x2="50.605" y2="90.2" width="1.016" layer="16"/>
+<wire x1="50.605" y1="90.2" x2="50.605" y2="90.24" width="1.016" layer="16"/>
 </signal>
 <signal name="N$2">
@@
 <wire x1="124.7714" y1="92.3286" x2="124.7714" y2="84.5" width="0.254" layer="1"/>
 <wire x1="124" y1="93.1" x2="124.7714" y2="92.3286" width="0.254" layer="1"/>
-<wire x1="124.7714" y1="84.5" x2="124.75" y2="84.5" width="0" layer="19" extent="1-1"/>
+<wire x1="124.7714" y1="84.5" x2="124.75" y2="84.5" width="0.254" layer="1"/>
 </signal>
 <signal name="RF_P">
@@
 <wire x1="125.2286" y1="92.3286" x2="125.2286" y2="84.5" width="0.254" layer="1"/>
 <wire x1="126" y1="93.1" x2="125.2286" y2="92.3286" width="0.254" layer="1"/>
-<wire x1="125.2286" y1="84.5" x2="125.25" y2="84.5" width="0" layer="19" extent="1-1"/>
+<wire x1="125.25" y1="84.5" x2="125.2286" y2="84.5" width="0.254" layer="1"/>
 </signal>
 <signal name="VCUTOFF">
