File: Controller/Eagle/Projects/Controller/controller_v6.brd (EAGLE design)
At the start: 250 x 115 mm, 74 parts, among them J2 AVR_SPI_PRG_6NS, J3 GIMBAL_3PIN, J4 GIMBAL_3PIN, J5 GIMBAL_3PIN, J6 GIMBAL_3PIN, U2 ATMEGA128RFA1, Y1 32.768kHz, Y2 16MHz

Commit message: Accidentally committed these
Routing:
- net GND: track 0.00 -> 1396.5 mm, vias 0 -> 23
- net 3.3V: track 0.00 -> 1124.9 mm, vias 0 -> 6
- net PE6: track 0.00 -> 136.6 mm
- net PD3/TXD1: track 0.00 -> 130.5 mm, vias 0 -> 2
- net PE7: track 0.00 -> 126.0 mm
- net RESET_N: track 0.00 -> 124.1 mm, vias 0 -> 5
- net PD2/RXD1: track 0.00 -> 105.6 mm, vias 0 -> 2
- net PB7: track 0.00 -> 94.8 mm
- net ADC3: track 0.00 -> 87.6 mm, vias 0 -> 2
- net PB4: track 0.00 -> 87.0 mm, vias 0 -> 2
- net PD0/I2C_SCL: track 0.00 -> 86.1 mm, vias 0 -> 2
- net ADC0: track 0.00 -> 82.5 mm, vias 0 -> 1
- net PB6: track 0.00 -> 79.1 mm
- net PD1/I2C_SDA: track 0.00 -> 76.1 mm, vias 0 -> 2
- net ADC2: track 0.00 -> 73.4 mm, vias 0 -> 2
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
Commit message: Moved the controller code to a more sensible place
Routing:
- net GND: track 1396.5 -> 0.00 mm, vias 23 -> 0
- net 3.3V: track 1124.9 -> 0.00 mm, vias 6 -> 0
- net PE6: track 136.6 -> 0.00 mm
- net PD3/TXD1: track 130.5 -> 0.00 mm, vias 2 -> 0
- net PE7: track 126.0 -> 0.00 mm
- net RESET_N: track 124.1 -> 0.00 mm, vias 5 -> 0
- net PD2/RXD1: track 105.6 -> 0.00 mm, vias 2 -> 0
- net PB7: track 94.8 -> 0.00 mm
- net ADC3: track 87.6 -> 0.00 mm, vias 2 -> 0
- net PB4: track 87.0 -> 0.00 mm, vias 2 -> 0
- net PD0/I2C_SCL: track 86.1 -> 0.00 mm, vias 2 -> 0
- net ADC0: track 82.5 -> 0.00 mm, vias 1 -> 0
- net PB6: track 79.1 -> 0.00 mm
- net PD1/I2C_SDA: track 76.1 -> 0.00 mm, vias 2 -> 0
- net ADC2: track 73.4 -> 0.00 mm, vias 2 -> 0
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