File: Motor/motorboard_v1.2.brd (EAGLE design)
At the start: 42.9 x 34.3 mm, 10 parts, among them K1 653002114822, K2 653002114822, K3 653002114822, K4 653002114822, U1 ULN2003ANE4

Commit message: Update
Parts:
- added JP2: M02LOCK_LONGPADS, SparkFun-Connectors:1X02_LOCK_LONGPADS
- moved D1 10.5 mm to (34.3, 27.9)
- moved D2 10.5 mm to (34.3, 20.3)
- moved D3 10.5 mm to (34.3, 12.7)
- moved D4 10.5 mm to (34.3, 5.08)
- moved K1 10.5 mm to (34.3, 31.8)
- moved K2 10.5 mm to (34.3, 24.1)
- moved K3 10.5 mm to (34.3, 16.5)
- moved K4 10.5 mm to (34.3, 8.89)
- moved JP1 9.25 mm to (2.54, 5.08)
- moved U1 9.25 mm to (20.3, 5.08)
Connections:
- net GND: now also JP2.1
- net N$1: now also JP2.2
Routing:
- net N$1: track 82.6 -> 117.1 mm
- net GND: track 17.8 -> 41.6 mm
- net N$9: track 18.3 -> 17.0 mm
- net N$8: track 16.2 -> 14.9 mm
- net N$7: track 18.3 -> 17.0 mm
Other:
- board text added: "- +"
