File: Motor/motorboard_v1.2.sch (EAGLE design)
At the start: 10 parts, among them K1 653002114822, K2 653002114822, K3 653002114822, K4 653002114822, U1 ULN2003ANE4

Commit message: Update
Parts:
- added JP2: M02LOCK_LONGPADS, SparkFun-Connectors:M02LOCK_LONGPADS
Connections:
- net GND: now also JP2.1
- net N$1: now also JP2.2
Changed lines of the file:
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@@
 <attribute name="OC_FARNELL" value="2295710"/>
 </part>
-<part name="P+1" library="ATmega128RFA1-DevBoard" deviceset="3.3V" device=""/>
 <part name="GND1" library="supply1" deviceset="GND" device=""/>
+<part name="GND2" library="supply1" deviceset="GND" device=""/>
+<part name="JP2" library="SparkFun-Connectors" deviceset="M02" device="LOCK_LONGPADS"/>
 </parts>
 <sheets>
@@
 <attribute name="MPN" x="111.76" y="25.4" size="1.778" layer="96" display="off"/>
 </instance>
-<instance part="P+1" gate="G$1" x="-45.72" y="-22.86"/>
 <instance part="GND1" gate="1" x="-17.78" y="-30.48"/>
+<instance part="GND2" gate="1" x="5.08" y="-58.42"/>
+<instance part="JP2" gate="G$1" x="-5.08" y="-53.34" smashed="yes">
+<attribute name="NAME" x="-7.62" y="-47.498" size="1.778" layer="95"/>
+</instance>
 </instances>
 <busses>
@@
 <wire x1="-30.48" y1="-22.86" x2="-25.4" y2="-22.86" width="0.1524" layer="91"/>
 <wire x1="-25.4" y1="-22.86" x2="-25.4" y2="-35.56" width="0.1524" layer="91"/>
-<wire x1="-25.4" y1="-35.56" x2="33.02" y2="-35.56" width="0.1524" layer="91"/>
+<wire x1="-25.4" y1="-35.56" x2="5.08" y2="-35.56" width="0.1524" layer="91"/>
+<wire x1="5.08" y1="-35.56" x2="33.02" y2="-35.56" width="0.1524" layer="91"/>
 <wire x1="33.02" y1="-35.56" x2="33.02" y2="-25.4" width="0.1524" layer="91"/>
 <pinref part="U1" gate="A" pin="COM"/>
@@
 <pinref part="K4" gate="G$1" pin="1"/>
 <wire x1="106.68" y1="27.94" x2="109.22" y2="27.94" width="0.1524" layer="91"/>
+<wire x1="5.08" y1="-35.56" x2="5.08" y2="-50.8" width="0.1524" layer="91"/>
+<wire x1="5.08" y1="-50.8" x2="2.54" y2="-50.8" width="0.1524" layer="91"/>
+<pinref part="JP2" gate="G$1" pin="2"/>
 </segment>
 </net>
@@
 <pinref part="D4" gate="1" pin="A"/>
 <wire x1="111.76" y1="22.86" x2="109.22" y2="22.86" width="0.1524" layer="91"/>
-</segment>
-</net>
-<net name="3.3V" class="0">
-<segment>
-<pinref part="P+1" gate="G$1" pin="3.3V"/>
-<wire x1="-35.56" y1="-22.86" x2="-45.72" y2="-22.86" width="0.1524" layer="91"/>
 </segment>
 </net>
@@
 <wire x1="-17.78" y1="-27.94" x2="-17.78" y2="-25.4" width="0.1524" layer="91"/>
 </segment>
-</net>
+<segment>
+<pinref part="GND2" gate="1" pin="GND"/>
+<wire x1="2.54" y1="-53.34" x2="5.08" y2="-53.34" width="0.1524" layer="91"/>
+<wire x1="5.08" y1="-53.34" x2="5.08" y2="-55.88" width="0.1524" layer="91"/>
+<pinref part="JP2" gate="G$1" pin="1"/>
+</segment>
+</net>
