File: Master/master_jorge.sch (EAGLE design)
At the start: 51 parts, among them J1 ISP, K1 653002114822, K2 653002114822, K3 653002114822, K4 653002114822, U1 ATMEGA128RFA1, U3 ULN2003ADR, Y1 16MHz, Y2 32.768kHz

Commit message: DRC Check changes
Updating master_jorge board with some DRC checks.
Other:
- note added: "- Removed redundant diodes in Brushed Motot Driver - Changed Leds to 0603 package - Removed unesessary caps - Added Voltage testpoints in serial debuger. - CHECK Motor pin headers direction and motor direction. - TODO: Place Names in Silkscreen correctly."
- note removed: "- Removed redundant diodes in Brushed Motot Driver - Changed Leds to 0603 package - Removed unesessary caps - Added Voltage testpoints in serial debuger. - CHECK Motor pin headers direction and motor direction. - TODO: DRC for Layout - TODO: Place Names in Silkscreen correctly."
Changed lines of the file:
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@@
 <setting verticaltext="up"/>
 </settings>
-<grid distance="0.01" unitdist="inch" unit="inch" style="lines" multiple="1" display="no" altdistance="0.01" altunitdist="inch" altunit="inch"/>
+<grid distance="0.1" unitdist="inch" unit="inch" style="lines" multiple="1" display="no" altdistance="0.01" altunitdist="inch" altunit="inch"/>
 <layers>
 <layer number="1" name="Top" color="4" fill="1" visible="no" active="no"/>
@@
 - CHECK Motor pin headers direction
   and motor direction.
-- TODO: DRC for Layout
 - TODO: Place Names in Silkscreen correctly. </text>
 </plain>

Commit message: Updating Silkscreen
Updating silkscreen of master_jorge
Parts:
- renumbered U$1 to U2, U$3 to U4, U$6 to U5
Other:
- note added: "- Removed redundant diodes in Brushed Motot Driver - Changed Leds to 0603 package - Removed unesessary caps - Added Voltage testpoints in serial debuger. - TODO: CHECK Motor pin headers direction and motor direction. - TODO: Check manually all Wires vs Layout"
- note removed: "- Removed redundant diodes in Brushed Motot Driver - Changed Leds to 0603 package - Removed unesessary caps - Added Voltage testpoints in serial debuger. - CHECK Motor pin headers direction and motor direction. - TODO: Place Names in Silkscreen correctly."
