File: Master/master_jorge.sch (EAGLE design)
At the start: 51 parts, among them J1 ISP, K1 653002114822, K2 653002114822, K3 653002114822, K4 653002114822, U1 ATMEGA128RFA1, U2 TPS73633-DBVT, U3 ULN2003ADR, U4 LSM303D, U5 L3GD20H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

Commit message: Updating some designs
Parts:
- renumbered ARM to D3, BOT to D2, PWR to D1
Other:
- note added: "- Removed redundant diodes in Brushed Motot Driver - Changed Leds to 0603 package - Removed unesessary caps - Added Voltage testpoints in serial debuger. - TODO: CHECK Motor pin headers direction and motor direction. - TODO: Check manually all Wires vs Layout"
- note removed: "- Removed redundant diodes in Brushed Motot Driver - Changed Leds to 0603 package - Removed unesessary caps - Added Voltage testpoints in serial debuger."
Changed lines of the file:
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@@
 <part name="P+5" library="SparkFun-Aesthetics" deviceset="3.3V" device=""/>
 <part name="C15" library="resistor" deviceset="C-US" device="C0805" value="0.1uF"/>
-<part name="BOT" library="led" deviceset="LED" device="CHIPLED_0603" value="GREEN"/>
+<part name="D2" library="led" deviceset="LED" device="CHIPLED_0603" value="GREEN"/>
 <part name="C9" library="resistor" deviceset="C-US" device="C0805" value="0.75pF"/>
 <part name="GND13" library="SparkFun-Aesthetics" deviceset="GND" device=""/>
 <part name="C16" library="resistor" deviceset="C-US" device="C0805" value="JUMP"/>
 <part name="C17" library="resistor" deviceset="C-US" device="C0805" value="JUMP"/>
-<part name="ARM" library="led" deviceset="LED" device="CHIPLED_0603" value="GREEN"/>
+<part name="D3" library="led" deviceset="LED" device="CHIPLED_0603" value="GREEN"/>
 <part name="R5" library="resistor" deviceset="R-US_" device="R0805" value="330"/>
 <part name="R6" library="resistor" deviceset="R-US_" device="R0805" value="330"/>
@@
 <part name="SUPPLY3" library="supply2" deviceset="GND" device=""/>
 <part name="R2" library="resistor" deviceset="R-US_" device="R0805" value="330"/>
-<part name="PWR" library="led" deviceset="LED" device="CHIPLED_0603" value="RED"/>
+<part name="D1" library="led" deviceset="LED" device="CHIPLED_0603" value="RED"/>
 <part name="SUPPLY4" library="supply2" deviceset="GND" device=""/>
 <part name="FRAME1" library="frames" deviceset="FRAME_B_L" device="" value="NONE"/>
@@
 - Removed unesessary caps
 - Added Voltage testpoints in serial debuger.
-</text>
+- TODO: CHECK Motor pin headers direction
+  and motor direction.
+- TODO: Check manually all Wires vs Layout</text>
 </plain>
 <instances>
@@
 <instance part="P+5" gate="G$1" x="-226.86" y="218.04"/>
 <instance part="C15" gate="G$1" x="-214.16" y="205.34" rot="R90"/>
-<instance part="BOT" gate="G$1" x="-137.24" y="138.04" rot="MR0"/>
+<instance part="D2" gate="G$1" x="-137.24" y="138.04" rot="MR0"/>
 <instance part="C9" gate="G$1" x="-0.08" y="183.76" rot="MR180"/>
 <instance part="GND13" gate="1" x="-0.08" y="173.6" rot="MR0"/>
 <instance part="C16" gate="G$1" x="-30.56" y="191.38" rot="R90"/>
 <instance part="C17" gate="G$1" x="-33.1" y="171.06" rot="R270"/>
-<instance part="ARM" gate="G$1" x="-147.4" y="138.04" rot="MR0"/>
+<instance part="D3" gate="G$1" x="-147.4" y="138.04" rot="MR0"/>
 <instance part="R5" gate="G$1" x="-147.4" y="148.2" rot="R90"/>
 <instance part="R6" gate="G$1" x="-137.24" y="148.2" rot="R90"/>
@@
 <instance part="SUPPLY3" gate="GND" x="-233.68" y="269.24"/>
 <instance part="R2" gate="G$1" x="-172.72" y="269.24" rot="R90"/>
-<instance part="PWR" gate="G$1" x="-172.72" y="261.62" rot="MR0"/>
+<instance part="D1" gate="G$1" x="-172.72" y="261.62" rot="MR0"/>
 <instance part="SUPPLY4" gate="GND" x="-172.72" y="254"/>
 <instance part="FRAME1" gate="G$1" x="-284.48" y="25.4"/>
@@
 </segment>
 <segment>
-<pinref part="ARM" gate="G$1" pin="C"/>
+<pinref part="D3" gate="G$1" pin="C"/>
 <pinref part="GND30" gate="1" pin="GND"/>
 <wire x1="-147.4" y1="132.96" x2="-147.4" y2="130.42" width="0.1524" layer="91"/>
 </segment>
 <segment>
-<pinref part="BOT" gate="G$1" pin="C"/>
+<pinref part="D2" gate="G$1" pin="C"/>
 <pinref part="GND31" gate="1" pin="GND"/>
 <wire x1="-137.24" y1="132.96" x2="-137.24" y2="130.42" width="0.1524" layer="91"/>
@@
 </segment>
 <segment>
-<pinref part="PWR" gate="G$1" pin="C"/>
+<pinref part="D1" gate="G$1" pin="C"/>
 <pinref part="SUPPLY4" gate="GND" pin="GND"/>
 </segment>
@@
 <net name="N$8" class="0">
 <segment>
-<pinref part="ARM" gate="G$1" pin="A"/>
+<pinref part="D3" gate="G$1" pin="A"/>
 <pinref part="R5" gate="G$1" pin="1"/>
 <wire x1="-147.4" y1="143.12" x2="-147.4" y2="140.58" width="0.1524" layer="91"/>
@@
 <net name="N$13" class="0">
 <segment>
-<pinref part="BOT" gate="G$1" pin="A"/>
+<pinref part="D2" gate="G$1" pin="A"/>
 <pinref part="R6" gate="G$1" pin="1"/>
 <wire x1="-137.24" y1="143.12" x2="-137.24" y2="140.58" width="0.1524" layer="91"/>
@@
 <segment>
 <pinref part="R2" gate="G$1" pin="1"/>
-<pinref part="PWR" gate="G$1" pin="A"/>
-</segment>
-</net>
+<pinref part="D1" gate="G$1" pin="A"/>
+</segment>
+</net>
