File: Master/master_jorge.brd (EAGLE design)
At the start: 44.7 x 35.8 mm, 51 parts, among them J1 ISP, K1 653002114822, K2 653002114822, K3 653002114822, K4 653002114822, U1 ATMEGA128RFA1, U2 TPS73633-DBVT, U3 ULN2003ADR, U4 LSM303D, U5 L3GD20H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

Commit message: Updating some designs
Parts:
- renumbered ARM to D3, BOT to D2, PWR to D1
Changed lines of the file:
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@@
 <wire x1="44.196" y1="39.37" x2="44.196" y2="37.592" width="0.6096" layer="51"/>
 <text x="-17.272" y="18.288" size="1.778" layer="51">1.41 inch
-35.81 mm</text>
+35.81  mm</text>
 <text x="17.018" y="41.91" size="1.778" layer="51">1.76 inch
 44.70 mm</text>
@@
 <attribute name="VALUE" x="27.1526" y="26.2128" size="1.27" layer="27" rot="R90"/>
 </element>
-<element name="PWR" library="led" package="CHIPLED_0603" value="RED" x="34.0106" y="3.2258" smashed="yes" rot="R180">
+<element name="D1" library="led" package="CHIPLED_0603" value="RED" x="34.0106" y="3.2258" smashed="yes" rot="R180">
 <attribute name="NAME" x="33.5042" y="0.9456" size="0.8128" layer="21"/>
 <attribute name="VALUE" x="32.1056" y="4.4958" size="1.27" layer="27" rot="R270"/>
 </element>
-<element name="BOT" library="led" package="CHIPLED_0603" value="GREEN" x="31.4706" y="3.2258" smashed="yes" rot="R180">
-<attribute name="NAME" x="30.3962" y="1.0056" size="0.8128" layer="21"/>
+<element name="D2" library="led" package="CHIPLED_0603" value="GREEN" x="31.4706" y="3.2258" smashed="yes" rot="R180">
+<attribute name="NAME" x="30.9042" y="1.0056" size="0.8128" layer="21"/>
 <attribute name="VALUE" x="29.5656" y="4.4958" size="1.27" layer="27" rot="R270"/>
 </element>
-<element name="ARM" library="led" package="CHIPLED_0603" value="GREEN" x="28.9306" y="3.2258" smashed="yes" rot="R180">
-<attribute name="NAME" x="27.1342" y="1.0656" size="0.8128" layer="21"/>
+<element name="D3" library="led" package="CHIPLED_0603" value="GREEN" x="28.9306" y="3.2258" smashed="yes" rot="R180">
+<attribute name="NAME" x="28.4042" y="1.0656" size="0.8128" layer="21"/>
 <attribute name="VALUE" x="27.0256" y="4.4958" size="1.27" layer="27" rot="R270"/>
 </element>
@@
 <attribute name="SUPPLIER" value="TEXAS INSTRUMENTS" x="16.4846" y="3.2258" size="1.778" layer="27" rot="R270" display="off"/>
 <attribute name="OC_FARNELL" value="1470513" x="16.4846" y="3.2258" size="1.778" layer="27" rot="R270" display="off"/>
-<attribute name="NAME" x="26.168" y="7.6168" size="0.8128" layer="21" ratio="10" rot="SR0"/>
+<attribute name="NAME" x="14.738" y="3.2988" size="0.8128" layer="21" ratio="10" rot="SR0"/>
 <attribute name="VALUE" x="12.827" y="11.1506" size="2.0828" layer="27" ratio="10" rot="SR270"/>
 </element>
 <element name="Y1" library="SparkFun-FreqCtrl" package="CRYSTAL-SMD-5X3" value="16MHz" x="37.5666" y="5.2578" smashed="yes" rot="R90">
-<attribute name="NAME" x="37.2742" y="8.9196" size="0.8128" layer="21" rot="R180"/>
+<attribute name="NAME" x="37.7822" y="2.0616" size="0.8128" layer="21" rot="R180"/>
 <attribute name="VALUE" x="40.1066" y="2.7178" size="0.4064" layer="27" rot="R90"/>
 </element>
@@
 <contactref element="C11" pad="2"/>
 <contactref element="C9" pad="1"/>
-<contactref element="ARM" pad="C"/>
-<contactref element="BOT" pad="C"/>
+<contactref element="D3" pad="C"/>
+<contactref element="D2" pad="C"/>
 <contactref element="U1" pad="11"/>
 <contactref element="U1" pad="33"/>
@@
 <contactref element="C23" pad="2"/>
 <contactref element="U2" pad="2"/>
-<contactref element="PWR" pad="C"/>
+<contactref element="D1" pad="C"/>
 <contactref element="C18" pad="2"/>
 <contactref element="C19" pad="2"/>
@@
 </signal>
 <signal name="N$8">
-<contactref element="ARM" pad="A"/>
+<contactref element="D3" pad="A"/>
 <contactref element="R5" pad="1"/>
 <wire x1="28.9306" y1="6.1858" x2="28.9306" y2="3.9758" width="0.254" layer="1"/>
 </signal>
 <signal name="N$13">
-<contactref element="BOT" pad="A"/>
+<contactref element="D2" pad="A"/>
 <contactref element="R6" pad="1"/>
 <wire x1="31.4706" y1="6.1858" x2="31.4706" y2="3.9758" width="0.254" layer="1"/>
@@
 <contactref element="K3" pad="2"/>
 <via x="14.9606" y="2.4638" extent="1-16" drill="0.4064"/>
-<wire x1="22.8346" y1="3.2258" x2="22.8346" y2="4.4958" width="0.4064" layer="1"/>
-<wire x1="22.8346" y1="4.4958" x2="21.3106" y2="6.0198" width="0.4064" layer="1"/>
-<wire x1="21.3106" y1="6.0198" x2="20.2946" y2="6.0198" width="0.4064" layer="1"/>
-<wire x1="20.2946" y1="6.0198" x2="18.5166" y2="4.7498" width="0.4064" layer="1"/>
-<wire x1="18.5166" y1="4.7498" x2="14.9606" y2="4.7498" width="0.4064" layer="1"/>
-<wire x1="14.9606" y1="4.7498" x2="14.9606" y2="2.4638" width="0.4064" layer="1"/>
+<wire x1="22.8346" y1="3.2258" x2="22.8346" y2="4.4958" width="0.254" layer="1"/>
+<wire x1="22.8346" y1="4.4958" x2="21.3106" y2="6.0198" width="0.254" layer="1"/>
+<wire x1="21.3106" y1="6.0198" x2="20.2946" y2="6.0198" width="0.254" layer="1"/>
+<wire x1="20.2946" y1="6.0198" x2="18.5166" y2="4.7498" width="0.254" layer="1"/>
+<wire x1="18.5166" y1="4.7498" x2="14.9606" y2="4.7498" width="0.254" layer="1"/>
+<wire x1="14.9606" y1="4.7498" x2="14.9606" y2="2.4638" width="0.254" layer="1"/>
 <wire x1="14.9606" y1="2.4638" x2="2.3776" y2="2.4638" width="0.4064" layer="16"/>
 <wire x1="2.3776" y1="2.4638" x2="2.2606" y2="2.3468" width="0.4064" layer="16"/>
@@
 <signal name="N$2">
 <contactref element="R2" pad="1"/>
-<contactref element="PWR" pad="A"/>
+<contactref element="D1" pad="A"/>
 <wire x1="34.0106" y1="6.1858" x2="34.0106" y2="3.9758" width="0.254" layer="1"/>
 </signal>
