File: Master/master_jorge3.brd (EAGLE design)
At the start: 73.4 x 73.4 mm, 51 parts, among them J1 ISP, K1 653002114822, K2 653002114822, K3 653002114822, K4 653002114822, U1 ATMEGA128RFA1, U2 TPS73633-DBVT, U3 ULN2003ADR, U4 LSM303D, U5 L3GD20H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

Commit message: Updating some designs
Other:
- board size 73.4 x 73.4 mm -> 71.7 x 73.6 mm
- board text added: "1.4 inch 35.56 mm"
- board text added: "2.82 inch 71.70 mm"
- board text added: "2.90 inch 73.66 mm"
- board text removed: "1.76 inch 44.70 mm"
