File: Master/master_muhsin_v4.brd (EAGLE design)
At the start: 61 x 61 mm, 51 parts, among them J1 ISP, K1 653002114822, K2 653002114822, K3 653002114822, K4 653002114822, U1 ATMEGA128RFA1, U2 TPS73633-DBVT, U3 ULN2003ADR, U4 LSM303D, U5 L3GD20H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

Commit message: Update
Parts:
- moved C11 5.08 mm to (13.2, 43.5)
- moved C14 5.08 mm to (20.9, 39.4)
- moved C16 5.08 mm to (21.0, 55.1)
- moved C17 5.08 mm to (10.8, 43.5)
- moved C18 5.08 mm to (18.8, 39.4)
- moved C19 5.08 mm to (22.6, 39.4)
- moved C20 5.08 mm to (15.3, 39.4)
- moved C21 5.08 mm to (17.0, 39.4)
- moved C8 5.08 mm to (25.8, 52.4)
- moved C9 5.08 mm to (16.3, 43.5)
- moved Y2 5.08 mm to (21.8, 50.9)
- moved C12 5.08 mm to (22.5, 19.7)
- moved JP9 5.08 mm to (45.6, 36.0)
- moved U4 5.08 mm to (20.4, 35.0)
- moved C3 5.08 mm to (17.5, 12.8)
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Other:
- board size 61 x 61 mm -> 72.4 x 71.1 mm
