File: Master/master_taylor.sch (EAGLE design)
At the start: 46 parts, among them J1 ISP, K1 653002114822, K2 653002114822, K3 653002114822, K4 653002114822, U1 ATMEGA128RFA1, U2 TPS73633-DBVT, U3 ULN2003ADR, Y1 16MHz, Y2 32.768kHz

Commit message: IMU has name and value
Parts:
- removed C15: 0.1uF, resistor:C-USC0805
- removed C7, C8: 12pF, resistor:C-USC0805
- removed Y2: 32.768kHz, SparkFun-FreqCtrl:CRYSTAL32-SMD
Connections:
- removed net N$5: C7.1, U1.PG4(TOSC1), Y2.1
- removed net N$6: C8.1, U1.PG3(TOSC2), Y2.2
- new net N$14: J1.2
- new net N$9: JP9.4
- net 3.3V: no longer J1.2, JP9.4
- net DTR: no longer C15.1
- net GND: no longer C7.2, C8.2
- net RESET: no longer C15.2
Changed lines of the file:
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@@
 <setting verticaltext="up"/>
 </settings>
-<grid distance="0.1" unitdist="inch" unit="inch" style="lines" multiple="1" display="yes" altdistance="0.01" altunitdist="inch" altunit="inch"/>
+<grid distance="0.1" unitdist="inch" unit="inch" style="lines" multiple="1" display="no" altdistance="0.01" altunitdist="inch" altunit="inch"/>
 <layers>
 <layer number="1" name="Top" color="4" fill="1" visible="no" active="no"/>
@@
 <part name="GND6" library="SparkFun-Aesthetics" deviceset="GND" device=""/>
 <part name="GND7" library="SparkFun-Aesthetics" deviceset="GND" device=""/>
-<part name="Y2" library="SparkFun-FreqCtrl" deviceset="CRYSTAL" device="32-SMD" value="32.768kHz"/>
-<part name="C7" library="resistor" deviceset="C-US" device="C0805" value="12pF"/>
-<part name="C8" library="resistor" deviceset="C-US" device="C0805" value="12pF"/>
-<part name="GND8" library="SparkFun-Aesthetics" deviceset="GND" device=""/>
-<part name="GND9" library="SparkFun-Aesthetics" deviceset="GND" device=""/>
 <part name="B1" library="SparkFun-RF" deviceset="BALUN" device="0805" value="748421245"/>
 <part name="C11" library="resistor" deviceset="C-US" device="C0805" value="22pF"/>
@@
 <part name="P+7" library="SparkFun-Aesthetics" deviceset="3.3V" device=""/>
 <part name="P+9" library="SparkFun-Aesthetics" deviceset="3.3V" device=""/>
-<part name="P+10" library="SparkFun-Aesthetics" deviceset="3.3V" device=""/>
 <part name="S1" library="SparkFun-Electromechanical" deviceset="SWITCH-MOMENTARY-2" device="SMD" value=""/>
 <part name="GND16" library="SparkFun-Aesthetics" deviceset="GND" device=""/>
 <part name="JP9" library="SparkFun-Connectors" deviceset="FTDI_BASIC" device="PTH" value="FTDI"/>
 <part name="GND25" library="SparkFun-Aesthetics" deviceset="GND" device=""/>
-<part name="P+5" library="SparkFun-Aesthetics" deviceset="3.3V" device=""/>
-<part name="C15" library="resistor" deviceset="C-US" device="C0805" value="0.1uF"/>
 <part name="D2" library="led" deviceset="LED" device="CHIPLED_0603" value="GREEN"/>
 <part name="C9" library="resistor" deviceset="C-US" device="C0805" value="0.75pF"/>
@@
 <instance part="GND6" gate="1" x="-40.72" y="138.04" rot="MR0"/>
 <instance part="GND7" gate="1" x="-50.88" y="138.04" rot="MR0"/>
-<instance part="Y2" gate="G$1" x="-139.78" y="117.72" smashed="yes" rot="MR0">
-<attribute name="NAME" x="-141.05" y="115.434" size="1.778" layer="95" rot="MR0"/>
-<attribute name="VALUE" x="-141.304" y="117.974" size="1.778" layer="96" rot="MR0"/>
-</instance>
-<instance part="C7" gate="G$1" x="-134.7" y="110.1" rot="MR0"/>
-<instance part="C8" gate="G$1" x="-144.86" y="110.1" rot="MR0"/>
-<instance part="GND8" gate="1" x="-134.7" y="102.48" rot="MR0"/>
-<instance part="GND9" gate="1" x="-144.86" y="102.48" rot="MR0"/>
 <instance part="B1" gate="G$1" x="-15.32" y="183.76" smashed="yes" rot="MR0">
 <attribute name="VALUE" x="-10.24" y="174.108" size="1.778" layer="96" rot="MR90"/>
@@
 <instance part="P+7" gate="G$1" x="-63.58" y="204.08" rot="MR0"/>
 <instance part="P+9" gate="G$1" x="-160.14" y="210.32" rot="MR0"/>
-<instance part="P+10" gate="G$1" x="-224.08" y="159.4"/>
 <instance part="S1" gate="G$1" x="-209.14" y="152.78" rot="R270"/>
 <instance part="GND16" gate="1" x="-209.14" y="142.62"/>
 <instance part="JP9" gate="G$1" x="-234.48" y="200.26" rot="MR180"/>
 <instance part="GND25" gate="1" x="-226.86" y="187.56"/>
-<instance part="P+5" gate="G$1" x="-226.86" y="218.04"/>
-<instance part="C15" gate="G$1" x="-214.16" y="205.34" rot="R90"/>
 <instance part="D2" gate="G$1" x="-137.24" y="138.04" rot="MR0"/>
 <instance part="C9" gate="G$1" x="-0.08" y="183.76" rot="MR180"/>
@@
 </segment>
 <segment>
-<pinref part="C7" gate="G$1" pin="2"/>
-<pinref part="GND8" gate="1" pin="GND"/>
-</segment>
-<segment>
-<pinref part="C8" gate="G$1" pin="2"/>
-<pinref part="GND9" gate="1" pin="GND"/>
-</segment>
-<segment>
 <pinref part="U1" gate="G$1" pin="AVSS_RFN"/>
 <wire x1="-68.66" y1="171.06" x2="-63.58" y2="171.06" width="0.1524" layer="91"/>
@@
 </segment>
 </net>
-<net name="N$5" class="0">
-<segment>
-<pinref part="C7" gate="G$1" pin="1"/>
-<wire x1="-134.7" y1="112.64" x2="-134.7" y2="117.72" width="0.1524" layer="91"/>
-<pinref part="U1" gate="G$1" pin="PG4(TOSC1)"/>
-<wire x1="-124.54" y1="117.72" x2="-134.7" y2="117.72" width="0.1524" layer="91"/>
-<pinref part="Y2" gate="G$1" pin="1"/>
-<wire x1="-137.24" y1="117.72" x2="-134.7" y2="117.72" width="0.1524" layer="91"/>
-<junction x="-134.7" y="117.72"/>
-</segment>
-</net>
-<net name="N$6" class="0">
-<segment>
-<pinref part="C8" gate="G$1" pin="1"/>
-<wire x1="-144.86" y1="112.64" x2="-144.86" y2="117.72" width="0.1524" layer="91"/>
-<pinref part="U1" gate="G$1" pin="PG3(TOSC2)"/>
-<wire x1="-144.86" y1="117.72" x2="-144.86" y2="120.26" width="0.1524" layer="91"/>
-<wire x1="-144.86" y1="120.26" x2="-124.54" y2="120.26" width="0.1524" layer="91"/>
-<pinref part="Y2" gate="G$1" pin="2"/>
-<wire x1="-142.32" y1="117.72" x2="-144.86" y2="117.72" width="0.1524" layer="91"/>
-<junction x="-144.86" y="117.72"/>
-</segment>
-</net>
 <net name="RFN" class="0">
 <segment>
@@
 <wire x1="-209.14" y1="160.4" x2="-206.6" y2="160.4" width="0.1524" layer="91"/>
 </segment>
-<segment>
-<pinref part="C15" gate="G$1" pin="2"/>
-<label x="-209.08" y="205.34" size="1.27" layer="95" xref="yes"/>
-<junction x="-209.08" y="205.34"/>
-</segment>
 </net>
 <net name="PE4" class="0">
@@
 <wire x1="-160.14" y1="210.32" x2="-160.14" y2="205.24" width="0.1524" layer="91"/>
 <pinref part="P+9" gate="G$1" pin="3.3V"/>
-</segment>
-<segment>
-<pinref part="J1" gate="G$1" pin="2"/>
-<wire x1="-226.62" y1="154.32" x2="-224.08" y2="154.32" width="0.1524" layer="91"/>
-<wire x1="-224.08" y1="154.32" x2="-224.08" y2="159.4" width="0.1524" layer="91"/>
-<pinref part="P+10" gate="G$1" pin="3.3V"/>
-</segment>
-<segment>
-<pinref part="JP9" gate="G$1" pin="4"/>
-<wire x1="-229.4" y1="197.72" x2="-226.86" y2="197.72" width="0.1524" layer="91"/>
-<wire x1="-226.86" y1="197.72" x2="-226.86" y2="218.04" width="0.1524" layer="91"/>
-<pinref part="P+5" gate="G$1" pin="3.3V"/>
 </segment>
 <segment>
@@
 <segment>
 <pinref part="JP9" gate="G$1" pin="1"/>
-<pinref part="C15" gate="G$1" pin="1"/>
 <wire x1="-216.7" y1="205.34" x2="-229.4" y2="205.34" width="0.1524" layer="91"/>
 </segment>
@@
 </segment>
 </net>
+<net name="N$9" class="0">
+<segment>
+<pinref part="JP9" gate="G$1" pin="4"/>
+<wire x1="-229.4" y1="197.72" x2="-226.86" y2="197.72" width="0.1524" layer="91"/>
+<wire x1="-226.86" y1="197.72" x2="-226.86" y2="218.04" width="0.1524" layer="91"/>
+</segment>
+</net>
+<net name="N$14" class="0">
+<segment>
+<pinref part="J1" gate="G$1" pin="2"/>
+<wire x1="-226.62" y1="154.32" x2="-224.08" y2="154.32" width="0.1524" layer="91"/>
+<wire x1="-224.08" y1="154.32" x2="-224.08" y2="159.4" width="0.1524" layer="91"/>
+</segment>
+</net>
