File: Master/master_brandon.brd (EAGLE design)
At the start: 84.3 x 69.3 mm, 58 parts, among them J1 ISP, K1 653002114822, K2 653002114822, K3 653002114822, K4 653002114822, U1 ATMEGA128RFA1, U3 ULN2003ANE4, Y1 16MHz, Y2 32.768kHz

Commit message: worked on my layout.  The rest can be auto-routed
Parts:
- moved D5 19.2 mm to (52.1, 54.3)
- moved K2 18.6 mm to (64.5, 54.3)
- moved U3 18.0 mm to (61.8, 5.89), turned to 0 degrees
- moved JP3 17.2 mm to (68.6, 20.9)
- moved R2 13.2 mm to (67.5, 14.4)
- moved C10 11.9 mm to (57.5, 36.5)
- moved K3 9.80 mm to (3.35, 53.9)
- moved R4 9.42 mm to (50.8, 38.1)
- moved R9 9.42 mm to (59.7, 48.6)
- moved U$6 9.42 mm to (62.6, 44.5)
- moved C14 9.42 mm to (50.2, 49.9)
- moved C20 9.42 mm to (54.4, 45.2)
- moved R7 9.42 mm to (48.8, 38.1)
- moved R8 9.42 mm to (56.4, 48.6)
- moved U$3 9.42 mm to (50.4, 44.7)
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Routing:
- net GND: track 45.5 -> 177.0 mm
- net RESET: track 0.00 -> 14.4 mm
- net N$5: track 0.00 -> 13.4 mm
- net N$6: track 0.00 -> 13.2 mm
- net N$4: track 0.00 -> 8.73 mm
- net N$3: track 0.00 -> 8.30 mm
- net RFANT: track 0.00 -> 6.27 mm
- net 3.3V: track 41.1 -> 46.7 mm
- net SDA: track 26.6 -> 31.8 mm
- net PB5: track 0.00 -> 5.07 mm
- net AVDD: track 0.00 -> 4.65 mm
- net PB4: track 0.00 -> 4.65 mm
- net PE4: track 0.00 -> 4.57 mm
- net PB6: track 0.00 -> 4.44 mm
- net N$7: track 0.00 -> 4.13 mm
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Other:
- board size 84.3 x 69.3 mm -> 76.8 x 60.3 mm

Commit message: Continued working on my layout
Parts:
- moved K3 85.4 mm to (70.2, 0.73), turned to 90 degrees
- moved D6 71.5 mm to (61.5, 0.06)
- moved K4 64.0 mm to (2.68, 1.55), turned to 270 degrees
- moved K1 52.6 mm to (3.40, 54.6), turned to 90 degrees
- moved D4 52.5 mm to (12.6, 53.3)
- moved D7 46.9 mm to (9.02, 5.35), turned to 90 degrees
- moved D1 24.6 mm to (52.9, 28.5)
- moved R2 24.3 mm to (53.4, 34.2)
- moved D5 9.10 mm to (61.2, 54.4)
- moved JP3 8.60 mm to (71.2, 12.7), turned to 270 degrees
- moved K2 5.82 mm to (70.2, 53.1), turned to 90 degrees
- moved S1 5.25 mm to (4.24, 42.2)
- moved R1 3.05 mm to (11.9, 42.7)
Routing:
- net VCC: track 0.00 -> 211.8 mm
- net N$29: track 0.00 -> 115.1 mm
- net N$32: track 0.00 -> 80.3 mm
- net N$30: track 0.00 -> 55.8 mm
- net GND: track 177.0 -> 225.9 mm
- net N$31: track 0.00 -> 26.9 mm

Commit message: updated Brandon's Master
Parts:
- U3: value ULN2003ANE4 -> ULN2003ADR; device Texas Instruments_By_element14_Batch_1:DIP254P762X508-16 -> Texas Instruments_By_element14_Batch_1:SOIC127P600X175-16N
- moved U3 6.52 mm to (62.1, 12.4)
Connections:
- removed net VDD: C10.1, JP1.1, R2.2, U$1.5
- net 3.3V: now also C10.1, JP1.1, R2.2, U$1.5
Routing:
- net VCC: track 211.8 -> 255.9 mm, vias 0 -> 1
- net N$26: track 80.3 -> 93.6 mm
- net GND: track 225.9 -> 218.0 mm, vias 2 -> 4
- net N$24: track 55.8 -> 53.6 mm
- net N$29: track 115.1 -> 117.2 mm

Commit message: Finished routing my board
Routing:
- net 3.3V: track 46.7 -> 243.2 mm, vias 0 -> 2
- net GND: track 218.0 -> 354.5 mm
- net RESET: track 14.0 -> 104.9 mm, vias 0 -> 3
- net PE3: track 3.15 -> 67.8 mm, vias 0 -> 2
- net PE4: track 4.57 -> 63.9 mm, vias 0 -> 2
- net SCL: track 29.2 -> 62.0 mm, vias 2 -> 3
- net PB4: track 4.65 -> 36.5 mm
- net RX0: track 0.00 -> 30.1 mm
- net SDA: track 31.8 -> 61.9 mm, vias 2 -> 3
- net MISO: track 3.99 -> 30.1 mm
- net PB5: track 5.07 -> 28.0 mm, vias 0 -> 2
- net SCK: track 2.63 -> 24.5 mm, vias 0 -> 1
- net MOSI: track 3.37 -> 23.8 mm
- net TX0: track 0.00 -> 20.2 mm
- net N$13: track 0.00 -> 16.5 mm
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
Commit message: Updated master_brandon
Parts:
- removed C19, C21: 0.1uF, SparkFun-Capacitors:0805
- removed C20: 10uF, SparkFun-Capacitors:0805
- removed C22: 10nF (25V), SparkFun-Capacitors:0805
- removed D4, D5, D6, D7: 1N4004, diode:DO41-10
- removed JP2: M01PTH, SparkFun:1X01
- removed R4, R7, R8, R9: 10k, SparkFun-Passives:0805
- removed U$3: LSM303D, IMU_parts:LGA16_3X3MM
- removed U$6: L3GD20H, IMU_parts:LGA16_3X3MM
- removed Y2: 32.768kHz, SparkFun-FreqCtrl:CRYSTAL-32KHZ-SMD
- added C24: 1uF, resistor:C0805
- added C25: 0.22uF, SparkFun-Capacitors:0603-CAP
- added C26: 4.7uF, SparkFun-Capacitors:0603-CAP
- added R10, R3: 10k, SparkFun-Passives:0805
- added U$2: LSM9DS0, IMU_parts:LGA-24
- C13: value 0.22uF -> 100nF; device SparkFun-Capacitors:0805 -> SparkFun-Capacitors:0603-CAP
- C14: value 4.7uF -> 10uF; device SparkFun-Capacitors:0805 -> SparkFun-Capacitors:EIA3528
- C15: value 0.1uF -> 1uF
- C18: device SparkFun-Capacitors:0805 -> resistor:C0805
- C7, C8: value 12pF -> 1uF
- D1: device Components:LED5MM -> master_devon:SML0603
- D2: value (none) -> RED; device Components:LED5MM -> led:CHIPLED_0603
- D3: value (none) -> WHITE; device Components:LED5MM -> led:CHIPLED_0603
- R5, R6: device resistor:R0805 -> SparkFun-Resistors:0603-RES
- U1: device SparkFun-DigitalIC:QFN-64 -> master_devon:QFN-64
- moved C14 52.3 mm to (18.3, 8.50)
- moved C18 48.6 mm to (74.8, 11.6), turned to 90 degrees
- moved C13 46.8 mm to (19.9, 4.80), turned to 270 degrees
- moved C8 44.7 mm to (62.2, 0.00), turned to 0 degrees
- moved C15 30.4 mm to (63.5, 54.5), turned to 0 degrees
- moved C7 23.0 mm to (7.60, 4.80)
- moved D2 11.3 mm to (44.9, 26.9)
- moved JP4 11.0 mm to (32.5, 15.8)
- moved C2 6.71 mm to (37.4, 6.29)
- moved D3 6.62 mm to (42.0, 26.9)
- moved R2 5.46 mm to (48.5, 31.8)
- moved D1 4.50 mm to (48.6, 27.0), turned to 90 degrees
- moved R6 2.86 mm to (44.9, 31.7)
- moved R5 0.82 mm to (41.9, 31.6)
Connections:
- removed net DTR: C15.1, JP9.DTR
- removed net N$12: C13.2, U$3.2
- removed net N$14: R4.1, U$3.8
- removed net N$15: R7.1, U$3.7
- removed net N$16: C14.2, U$3.15
- removed net N$17: R8.1, U$6.10
- removed net N$18: R9.1, U$6.9
- removed net N$19: C22.2, U$6.16
- new net N$22: C25.1, U$2.9
- new net N$23: R3.1, U$2.19
- net 3.3V: now also C13.1, C14.A, R10.2, R3.2, U$2.15, U$2.16, U$2.17, U$2.18; no longer C18.1, C19.1, C20.1, C21.1, J1.2, R4.2, R7.2, R8.2, R9.2, U$3.1, U$3.14, U$6.13, U$6.14
- net GND: now also C13.2, C14.C, C26.1, D1.C, D2.C, D3.C, U$2.2, U$2.22, U$2.23, U$2.3, U$2.4, U$2.5, U$2.6; no longer C14.1, C19.2, C20.2, C21.2, C22.1, C7.2, C8.2, D1.K, D2.K, D3.K, JP2.1, U$3.10, U$3.12, U$3.13, U$3.16, U$3.5, U$6.1, U$6.15, U$6.2, U$6.3, U$6.4, U$6.5, U$6.6
- net N$24: now also C15.2; no longer D5.A
- net N$25: now also C8.2; no longer D6.A
- net N$26: now also C7.2; no longer D7.A
- net N$29: now also C24.2; no longer D4.A
- net N$5: now also C26.2, U$2.7; no longer C7.1, U1.18, Y2.X1
- net N$6: now also C25.2, U$2.8; no longer C8.1, U1.17, Y2.X2
- net N$9: now also R10.1, U$2.20; no longer C13.1, U$3.3
- net PB4: now also U3.4; no longer U3.3
- net PB5: now also U3.3; no longer U3.2
- net PE3: now also U3.2; no longer U3.4
- net RESET: no longer C15.2
- net SCL: now also U$2.21; no longer U$3.4, U$6.12
- net SDA: now also U$2.24; no longer U$3.6, U$6.11
- net VCC: now also C15.1, C18.1, C24.1, C7.1, C8.1; no longer D4.C, D5.C, D6.C, D7.C
Routing:
- net SCL: track 62.0 -> 11.0 mm, vias 3 -> 2
- net SDA: track 61.9 -> 11.5 mm, vias 3 -> 2
- net GND: track 354.5 -> 308.2 mm, vias 4 -> 2
- net 3.3V: track 243.2 -> 199.3 mm
- net PE3: track 67.8 -> 30.7 mm
- net PE4: track 63.9 -> 32.8 mm
- net VCC: track 262.7 -> 290.5 mm, vias 1 -> 5
- net RESET: track 104.9 -> 77.4 mm, vias 3 -> 2
- net N$13: track 16.5 -> 3.24 mm
- net N$26: track 93.6 -> 80.7 mm
- net TX1: track 18.3 -> 6.68 mm, vias 1 -> 0
- net RX1: track 17.5 -> 5.88 mm, vias 1 -> 0
- net N$5: track 13.4 -> 2.70 mm
- net N$6: track 13.2 -> 4.37 mm
- net PB4: track 36.5 -> 28.3 mm
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Other:
- board text added: "BMW"
