File: Master/master_brandon.sch (EAGLE design)
At the start: 58 parts, among them J1 ISP, K1 653002114822, K2 653002114822, K3 653002114822, K4 653002114822, U1 ATMEGA128RFA1, U3 ULN2003ANE4, Y1 16MHz, Y2 32.768kHz

Commit message: updated Brandon's Master
Parts:
- U3: value ULN2003ANE4 -> ULN2003ADR; device Texas Instruments_By_element14_Batch_1:ULN2003ANE4 -> Texas Instruments_By_element14_Batch_1:ULN2003ADR
Connections:
- removed net VDD: C10.1, JP1.1, R2.2, U$1.OUT
- net 3.3V: now also C10.1, JP1.1, R2.2, U$1.OUT
- net GND: now also U3.E; no longer U3.GND
Other:
- moved on the sheet: U3

Commit message: Updated master_brandon
Parts:
- removed C19, C21: 0.1uF, SparkFun-Capacitors:CAP0805
- removed C20: 10uF, SparkFun-Capacitors:CAP0805
- removed C22: 10nF (25V), SparkFun-Capacitors:CAP0805
- removed D4, D5, D6, D7: 1N4004, diode:1N4004
- removed JP2: M01PTH, SparkFun:M01PTH
- removed R4, R7, R8, R9: 10k, SparkFun-Passives:RESISTOR0805-RES
- removed U$3: LSM303D, IMU_parts:LSM303D
- removed U$6: L3GD20H, IMU_parts:L3GD20H
- removed Y2: 32.768kHz, SparkFun-FreqCtrl:CRYSTAL32-SMD
- added C24: 1uF, resistor:C-USC0805
- added C25: 0.22uF, SparkFun-Capacitors:CAP0603-CAP
- added C26: 4.7uF, SparkFun-Capacitors:CAP0603-CAP
- added R10, R3: 10k, SparkFun-Passives:RESISTOR0805-RES
- added U$2: LSM9DS0, IMU_parts:LSM9DS0
- C13: value 0.22uF -> 100nF; device SparkFun-Capacitors:CAP0805 -> SparkFun-Capacitors:CAP0603-CAP
- C14: value 4.7uF -> 10uF; device SparkFun-Capacitors:CAP0805 -> SparkFun-Capacitors:10UF-20V-10%(TANT)
- C15: value 0.1uF -> 1uF
- C18: device SparkFun-Capacitors:CAP0805 -> resistor:C-USC0805
- C7, C8: value 12pF -> 1uF
- D1: device Components:LED5MM -> master_devon:LEDSML0603
- D2: value (none) -> RED; device Components:LED5MM -> led:LEDCHIPLED_0603
- D3: value (none) -> WHITE; device Components:LED5MM -> led:LEDCHIPLED_0603
- R5, R6: device resistor:R-US_R0805 -> SparkFun-Resistors:RESISTOR0603-RES
- U1: device SparkFun-DigitalIC:ATMEGA128RFA1 -> master_devon:ATMEGA128RFA1
Connections:
- removed net DTR: C15.1, JP9.1
- removed net N$12: C13.2, U$3.SETC
- removed net N$14: R4.1, U$3.CS
- removed net N$15: R7.1, U$3.SA0
- removed net N$16: C14.2, U$3.C1
- removed net N$17: R8.1, U$6.SA0
- removed net N$18: R9.1, U$6.CS
- removed net N$19: C22.2, U$6.CAP
- new net N$22: C25.1, U$2.SETP_XM
- new net N$23: R3.1, U$2.CS_G
- net 3.3V: now also C13.1, C14.+, R10.2, R3.2, U$2.VDD1, U$2.VDD2, U$2.VDD3, U$2.VDD_IO; no longer C18.1, C19.1, C20.1, C21.1, J1.2, R4.2, R7.2, R8.2, R9.2, U$3.VDD, U$3.VDD_IO, U$6.VDD, U$6.VDD_IO
- net GND: now also C13.2, C14.-, C26.1, U$2.GND1, U$2.GND2, U$2.RES2, U$2.RES3, U$2.RES4, U$2.SA0_G, U$2.SA0_XM; no longer C14.1, C19.2, C20.2, C21.2, C22.1, C7.2, C8.2, JP2.1, U$3.GND, U$3.GND1, U$3.GND2, U$3.GND3, U$3.RSRVD, U$6.DEN, U$6.GND, U$6.GND1, U$6.RSRV1, U$6.RSRV2, U$6.RSRV3, U$6.RSRV4
- net N$24: now also C15.2; no longer D5.A
- net N$25: now also C8.2; no longer D6.A
- net N$26: now also C7.2; no longer D7.A
- net N$29: now also C24.2; no longer D4.A
- net N$5: now also C26.2, U$2.C1_XM; no longer C7.1, U1.PG4(TOSC1), Y2.1
- net N$6: now also C25.2, U$2.SETC_XM; no longer C8.1, U1.PG3(TOSC2), Y2.2
- net N$9: now also R10.1, U$2.CS_XM; no longer C13.1, U$3.SETP
- net PB4: now also U3.4B; no longer U3.3B
- net PB5: now also U3.3B; no longer U3.2B
- net PE3: now also U3.2B; no longer U3.4B
- net RESET: no longer C15.2
- net SCL: now also U$2.SCL; no longer U$3.SCL, U$6.SCL
- net SDA: now also U$2.SDA; no longer U$3.SDA, U$6.SDA
- net VCC: now also C15.1, C18.1, C24.1, C7.1, C8.1; no longer D4.C, D5.C, D6.C, D7.C
Other:
- note removed: "L3GD20H (Gyroscope)"
- note removed: "LSM303D (Accelerometer)"
- moved on the sheet: C13, C15, C18, C7, C8, D2, D3, JP3, R5, R6
