File: Master/Devon/master_devon.routed.brd (EAGLE design)
At the start: 63.5 x 63.5 mm, 36 parts, among them J1 ISP, K1 653002114822, K2 653002114822, K3 653002114822, K4 653002114822, U1 ATMEGA128RFA1, U2 ULN2003ADR, Y1 16MHz

Commit message: Revert "Fixed main board"
This reverts commit e8d481ade4fad3f727996ef615af2e559dd81647.
Parts:
- moved JP3 45.4 mm to (48.3, 50.8), turned to 0 degrees
- moved U2 37.8 mm to (38.1, 50.8), turned to 90 degrees
- moved J1 27.8 mm to (-3.81, 33.0), turned to 90 degrees
- moved JP1 26.6 mm to (10.2, 12.7), turned to 90 degrees
- moved JP9 26.3 mm to (-5.08, -5.08)
- moved C10 17.9 mm to (24.1, 33.0)
- moved K1 16.6 mm to (-5.08, 53.3)
- moved C12 16.2 mm to (-5.08, 48.3)
- moved C3 13.0 mm to (19.1, 31.1)
- moved C2 12.7 mm to (33.0, 29.8)
- moved K2 12.1 mm to (-5.08, -12.7)
- moved K3 11.4 mm to (61.0, 53.3)
- moved C7 10.9 mm to (17.8, 43.2), turned to 270 degrees
- moved C14 10.8 mm to (61.0, 48.3)
- moved C8 9.44 mm to (22.9, -2.54)
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Connections:
- net PB4: no longer U2.4
- net PB5: now also U2.4; no longer U2.3
- net PE3: now also U2.1; no longer U2.2
- net PE4: now also U2.2; no longer U2.1
- net PE5: now also U2.3
Routing:
- net GND: track 0.00 -> 336.1 mm, vias 0 -> 2
- net VBATT: track 0.00 -> 220.5 mm
- net 3.3V: track 0.00 -> 128.3 mm, vias 0 -> 4
- net RESET: track 0.00 -> 125.1 mm, vias 0 -> 1
- net N$14: track 0.00 -> 97.7 mm, vias 0 -> 1
- net N$16: track 0.00 -> 88.8 mm
- net MOSI: track 0.00 -> 45.3 mm, vias 0 -> 1
- net TX0: track 0.00 -> 44.6 mm, vias 0 -> 1
- net VDD: track 0.00 -> 44.1 mm
- net RX0: track 0.00 -> 43.4 mm, vias 0 -> 1
- net PE4: track 0.00 -> 42.8 mm, vias 0 -> 2
- net N$12: track 0.00 -> 42.0 mm
- net PE5: track 0.00 -> 41.6 mm, vias 0 -> 2
- net SCK: track 0.00 -> 41.1 mm
- net MISO: track 0.00 -> 40.5 mm
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Other:
- board size 63.5 x 63.5 mm -> 76.2 x 76.2 mm

Commit message: Fixed main board
Hand routed some traces. Did some pin swapping. Now 2.5 x 2.5 inches.
Parts:
- moved JP3 45.4 mm to (7.62, 30.5), turned to 270 degrees
- moved U2 37.8 mm to (10.2, 25.4), turned to 180 degrees
- moved J1 27.8 mm to (8.89, 8.26), turned to 270 degrees
- moved JP1 26.6 mm to (27.3, 33.0), turned to 0 degrees
- moved JP9 26.3 mm to (20.3, -12.1)
- moved C10 17.9 mm to (41.3, 38.1)
- moved K1 16.6 mm to (6.99, 41.9)
- moved C12 16.2 mm to (6.99, 37.5)
- moved C3 13.0 mm to (27.9, 21.6)
- moved C2 12.7 mm to (22.9, 22.2)
- moved K2 12.1 mm to (6.99, -14.0)
- moved K3 11.4 mm to (61.6, 41.9)
- moved C7 10.9 mm to (16.5, 32.4), turned to 90 degrees
- moved C14 10.8 mm to (61.6, 37.5)
- moved C8 9.44 mm to (29.2, -9.53)
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Connections:
- net PB4: now also U2.4
- net PB5: now also U2.3; no longer U2.4
- net PE3: now also U2.2; no longer U2.1
- net PE4: now also U2.1; no longer U2.2
- net PE5: no longer U2.3
Routing:
- net GND: track 336.1 -> 0.00 mm, vias 2 -> 0
- net VBATT: track 220.5 -> 0.00 mm
- net 3.3V: track 128.3 -> 0.00 mm, vias 4 -> 0
- net RESET: track 125.1 -> 0.00 mm, vias 1 -> 0
- net N$14: track 97.7 -> 0.00 mm, vias 1 -> 0
- net N$16: track 88.8 -> 0.00 mm
- net MOSI: track 45.3 -> 0.00 mm, vias 1 -> 0
- net TX0: track 44.6 -> 0.00 mm, vias 1 -> 0
- net VDD: track 44.1 -> 0.00 mm
- net RX0: track 43.4 -> 0.00 mm, vias 1 -> 0
- net PE4: track 42.8 -> 0.00 mm, vias 2 -> 0
- net N$12: track 42.0 -> 0.00 mm
- net PE5: track 41.6 -> 0.00 mm, vias 2 -> 0
- net SCK: track 41.1 -> 0.00 mm
- net MISO: track 40.5 -> 0.00 mm
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Other:
- board size 76.2 x 76.2 mm -> 63.5 x 63.5 mm

Commit message: Made board smaller, fixed VDD->3.3V issue
Parts:
- moved C2 16.1 mm to (38.1, 27.3)
- moved C10 9.86 mm to (43.8, 28.6), turned to 180 degrees
- moved C3 5.08 mm to (22.9, 21.6)
- moved K3 4.49 mm to (62.2, 37.5)
- moved K1 4.44 mm to (6.99, 37.5)
- moved C14 3.86 mm to (62.2, 33.7)
- moved C12 3.81 mm to (6.99, 33.7)
Connections:
- removed net VDD: C10.+, C8.+, U$2.3
- net 3.3V: now also C10.+, C8.+, U$2.3
Routing:
- net GND: track 0.00 -> 264.2 mm
- net VBATT: track 0.00 -> 185.2 mm
- net 3.3V: track 0.00 -> 103.0 mm, vias 0 -> 5
- net RESET: track 0.00 -> 100.9 mm, vias 0 -> 3
- net N$16: track 0.00 -> 72.6 mm, vias 0 -> 1
- net N$15: track 0.00 -> 70.0 mm, vias 0 -> 1
- net N$14: track 0.00 -> 38.2 mm, vias 0 -> 1
- net PB7: track 0.00 -> 31.0 mm, vias 0 -> 2
- net SCK: track 0.00 -> 31.0 mm, vias 0 -> 1
- net PB6: track 0.00 -> 29.4 mm, vias 0 -> 2
- net MISO: track 0.00 -> 28.5 mm, vias 0 -> 1
- net TX0: track 0.00 -> 28.4 mm, vias 0 -> 1
- net N$12: track 0.00 -> 27.4 mm, vias 0 -> 1
- net RX0: track 0.00 -> 27.1 mm, vias 0 -> 1
- net MOSI: track 0.00 -> 26.4 mm, vias 0 -> 1
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Other:
- board size 63.5 x 63.5 mm -> 63.5 x 57.1 mm
- board text added: "+"
