File: Master/Jorge/master_jorge3newIMU.brd (EAGLE design)
At the start: 71.7 x 73.6 mm, 51 parts, among them J1 ISP, K1 653002114822, K2 653002114822, K3 653002114822, K4 653002114822, U1 ATMEGA128RFA1, U2 TPS73633-DBVT, U3 ULN2003ADR, U4 LSM303D, U5 L3GD20H, Y1 16MHz, Y2 32.768kHz

Commit message: Moving all my mess to a folder
Parts:
- removed C13: 0.22uF, SparkFun-Capacitors:0805
- removed C14: 4.7uF, SparkFun-Capacitors:0805
- removed C18, C20: 10uF, SparkFun-Capacitors:0805
- removed C19, C21: 0.1uF, SparkFun-Capacitors:0805
- removed C22: 10nF (25V), SparkFun-Capacitors:0805
- removed C7, C8: 12pF, resistor:C0805
- removed R4, R7, R8, R9: 10k, SparkFun-Passives:0805
- removed U5: L3GD20H, IMU_parts:LGA16_3X3MM
- removed Y2: 32.768kHz, SparkFun-FreqCtrl:CRYSTAL-32KHZ-SMD
- added C24: 10uF, SparkFun-Capacitors:0805
- added C25: 0.22uF, SparkFun-Capacitors:0805
- added C26: 4.7uF, SparkFun-Capacitors:0805
- added C4: 100nF, SparkFun-Capacitors:0805
- added R10, R3: 10k, SparkFun-Passives:0805
- ARM, BOT, PWR: device led:CHIPLED_0603 -> led:CHIP-LED0805
- JP1: value Debuger -> Debugger
- U4: value LSM303D -> LSM9DS0; device IMU_parts:LGA16_3X3MM -> IMU_parts:LGA-24
- moved C17 7.75 mm to (24.3, 26.4), turned to 270 degrees
- moved C11 6.65 mm to (21.3, 27.1), turned to 270 degrees
- moved A1 6.60 mm to (25.9, 32.4)
- moved C2 6.10 mm to (16.2, 27.1)
- moved C9 6.10 mm to (18.8, 27.1)
- moved C16 5.14 mm to (32.0, 26.3)
- moved C1 3.57 mm to (35.8, 26.8)
- moved B1 3.56 mm to (28.2, 28.6)
- moved U4 2.98 mm to (12.7, 18.6), turned to 0 degrees
- moved BOT 0.46 mm to (31.5, 3.68)
- moved ARM 0.43 mm to (29.0, 3.66)
- moved PWR 0.43 mm to (34.0, 3.66)
- moved R2 0.33 mm to (34.0, 7.37)
- moved R6 0.33 mm to (31.5, 7.37)
- moved R5 0.28 mm to (28.9, 7.32)
Connections:
- removed net N$12: C13.2, U4.2
- removed net N$14: R4.1, U4.8
- removed net N$15: R7.1, U4.7
- removed net N$16: C14.2, U4.15
- removed net N$17: R8.1, U5.10
- removed net N$18: R9.1, U5.9
- removed net N$19: C22.2, U5.16
- removed net N$5: C7.1, U1.18, Y2.X1
- removed net N$6: C8.1, U1.17, Y2.X2
- removed net N$9: C13.1, U4.3
- new net N$20: C26.2, U4.7
- new net N$21: C25.2, U4.8
- new net N$22: C25.1, U4.9
- new net N$23: R3.1, U4.19
- new net N$24: R10.1, U4.20
- net 3.3V: now also C24.1, C4.1, R10.2, R3.2, U4.15, U4.16, U4.17, U4.18; no longer C18.1, C19.1, C20.1, C21.1, R4.2, R7.2, R8.2, R9.2, U4.1, U4.14, U5.13, U5.14
- net GND: now also C24.2, C26.1, C4.2, U4.2, U4.22, U4.23, U4.3, U4.4, U4.6; no longer C14.1, C18.2, C19.2, C20.2, C21.2, C22.1, C7.2, C8.2, U4.10, U4.12, U4.13, U4.16, U5.1, U5.15, U5.2, U5.3, U5.4, U5.5, U5.6
- net SCL: now also U4.21; no longer U4.4, U5.12
- net SDA: now also U4.24; no longer U4.6, U5.11
Routing:
- net N$5: track 31.1 -> 0.00 mm, vias 2 -> 0
- net N$6: track 17.3 -> 0.00 mm, vias 2 -> 0
- net N$14: track 8.51 -> 0.00 mm
- net N$15: track 8.01 -> 0.00 mm
- net N$22: track 0.00 -> 6.72 mm
- net N$12: track 6.69 -> 0.00 mm
- net SCL: track 27.5 -> 20.9 mm, vias 3 -> 2
- net N$24: track 0.00 -> 6.41 mm
- net 3.3V: track 153.3 -> 159.2 mm
- net N$9: track 5.26 -> 0.00 mm
- net N$21: track 0.00 -> 5.04 mm
- net N$19: track 4.87 -> 0.00 mm
- net RFP: track 11.3 -> 6.91 mm
- net N$23: track 0.00 -> 4.08 mm
- net N$20: track 0.00 -> 3.73 mm
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
Commit message: Some updates
Some updates to my schematic and my board
Parts:
- added C13, C14, C7, C8: 1uF, resistor:C0805
- C24: device SparkFun-Capacitors:0805 -> rcl:C0805
- moved J1 4.37 mm to (40.4, 24.6)
- moved JP1 4.24 mm to (41.6, 11.3)
- moved Y1 3.20 mm to (39.4, 7.90), turned to 0 degrees
- moved S1 2.79 mm to (11.4, 31.4)
- moved C5 2.34 mm to (37.9, 12.9)
- moved C23 2.21 mm to (7.26, 6.71)
- moved C3 2.16 mm to (7.24, 13.5)
- moved C10 2.03 mm to (7.26, 8.81)
- moved C12 2.01 mm to (7.21, 11.1)
- moved C6 1.38 mm to (38.0, 15.2)
- moved C4 1.37 mm to (7.29, 16.2)
- moved C24 0.77 mm to (7.16, 21.8)
- moved R1 0.61 mm to (13.9, 26.5)
Connections:
- net 3.3V: no longer J1.2
- net N$29: now also C7.2
- net N$30: now also C8.2
- net N$31: now also C13.2
- net N$32: now also C14.2
- net VBAT: now also C13.1, C14.1, C7.1, C8.1
Routing:
- net VBAT: track 115.1 -> 133.1 mm
- net N$3: track 13.9 -> 21.3 mm
- net GND: track 233.2 -> 227.8 mm
- net N$29: track 18.7 -> 22.6 mm
- net MOSI: track 21.8 -> 25.6 mm
- net N$30: track 52.0 -> 55.8 mm
- net N$31: track 25.2 -> 28.8 mm
- net 3.3V: track 159.2 -> 156.3 mm, vias 7 -> 8
- net TX1: track 34.7 -> 31.8 mm
- net N$4: track 19.8 -> 17.0 mm
- net N$32: track 59.6 -> 62.2 mm
- net N$1: track 12.0 -> 13.8 mm
- net SCK: track 27.4 -> 28.9 mm
- net MISO: track 24.5 -> 25.5 mm
- net RESET: track 43.0 -> 43.8 mm
Other:
- board text added: "2.83 inch 71.88 mm"
- board text added: ">Info Board Name: UCSDQuadCop Part Number: 0 Number of Layers: 2 Dimension X= 2.83 inch Dimension Y= 2.90 inch Board Material Type: FR-4 Solder Mask Color: Red Silkscreen Color: White Finish Plating: HASAL Revision Number: 0"
- board text removed: "2.82 inch 71.70 mm"
- board text removed: ">Info Board Name: UCSDQuadCop Part Number: 0 Number of Layers: 2 Board Material Type: FR-4 Solder Mask Color: Red Silkscreen Color: White Finish Plating: HASAL Revision Number: 0"
