File: Master/Jorge/master_jorge3newIMU.sch (EAGLE design)
At the start: 51 parts, among them J1 ISP, K1 653002114822, K2 653002114822, K3 653002114822, K4 653002114822, U1 ATMEGA128RFA1, U2 TPS73633-DBVT, U3 ULN2003ADR, U4 LSM303D, U5 L3GD20H, Y1 16MHz, Y2 32.768kHz

Commit message: Moving all my mess to a folder
Parts:
- removed C13: 0.22uF, SparkFun-Capacitors:CAP0805
- removed C14: 4.7uF, SparkFun-Capacitors:CAP0805
- removed C18, C20: 10uF, SparkFun-Capacitors:CAP0805
- removed C19, C21: 0.1uF, SparkFun-Capacitors:CAP0805
- removed C22: 10nF (25V), SparkFun-Capacitors:CAP0805
- removed C7, C8: 12pF, resistor:C-USC0805
- removed R4, R7, R8, R9: 10k, SparkFun-Passives:RESISTOR0805-RES
- removed U5: L3GD20H, IMU_parts:L3GD20H
- removed Y2: 32.768kHz, SparkFun-FreqCtrl:CRYSTAL32-SMD
- added C24: 10uF, SparkFun-Capacitors:CAP0805
- added C25: 0.22uF, SparkFun-Capacitors:CAP0805
- added C26: 4.7uF, SparkFun-Capacitors:CAP0805
- added C4: 100nF, SparkFun-Capacitors:CAP0805
- added R10, R3: 10k, SparkFun-Passives:RESISTOR0805-RES
- ARM, BOT, PWR: device led:LEDCHIPLED_0603 -> led:LEDCHIP-LED0805
- JP1: value Debuger -> Debugger
- U4: value LSM303D -> LSM9DS0; device IMU_parts:LSM303D -> IMU_parts:LSM9DS0
Connections:
- removed net N$12: C13.2, U4.SETC
- removed net N$14: R4.1, U4.CS
- removed net N$15: R7.1, U4.SA0
- removed net N$16: C14.2, U4.C1
- removed net N$17: R8.1, U5.SA0
- removed net N$18: R9.1, U5.CS
- removed net N$19: C22.2, U5.CAP
- removed net N$5: C7.1, U1.PG4(TOSC1), Y2.1
- removed net N$6: C8.1, U1.PG3(TOSC2), Y2.2
- removed net N$9: C13.1, U4.SETP
- new net N$20: C26.2, U4.C1_XM
- new net N$21: C25.2, U4.SETC_XM
- new net N$22: C25.1, U4.SETP_XM
- new net N$23: R3.1, U4.CS_G
- new net N$24: R10.1, U4.CS_XM
- net 3.3V: now also C24.1, C4.1, R10.2, R3.2, U4.VDD1, U4.VDD2, U4.VDD3; no longer C18.1, C19.1, C20.1, C21.1, R4.2, R7.2, R8.2, R9.2, U4.VDD, U5.VDD, U5.VDD_IO
- net GND: now also C24.2, C26.1, C4.2, U4.RES2, U4.RES3, U4.RES4, U4.SA0_G, U4.SA0_XM; no longer C14.1, C18.2, C19.2, C20.2, C21.2, C22.1, C7.2, C8.2, U4.GND, U4.GND3, U4.RSRVD, U5.DEN, U5.GND, U5.GND1, U5.RSRV1, U5.RSRV2, U5.RSRV3, U5.RSRV4
- net SCL: no longer U5.SCL
- net SDA: no longer U5.SDA
Other:
- note added: "LSM9DS0 (Accelerometer, Gyroscope, Magnometer)"
- note added: "Serial Debugger"
- note removed: "L3GD20H (Gyroscope)"
- note removed: "LSM303D (Accelerometer)"
- note removed: "Serial Debuger"
- moved on the sheet: A1, ARM, B1, BOT, C1, C11, C16, C17, C2, C3, C5, C6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

Commit message: Some updates
Some updates to my schematic and my board
Parts:
- added C13, C14, C7, C8: 1uF, resistor:C-USC0805
- C24: device SparkFun-Capacitors:CAP0805 -> rcl:C-USC0805
Connections:
- net 3.3V: no longer J1.2
- net N$29: now also C7.2
- net N$30: now also C8.2
- net N$31: now also C13.2
- net N$32: now also C14.2
- net VBAT: now also C13.1, C14.1, C7.1, C8.1
Other:
- moved on the sheet: C24, K1, K2, K3, K4, U3
