File: Master/Jorge/REV1/master_jorge3newIMU.sch (EAGLE design)
At the start: 62 parts, among them J1 ISP, K1 653002114822, K2 653002114822, K3 653002114822, K4 653002114822, U1 ATMEGA128RFA1, U2 TPS73633-DBVT, U3 SI2366DS-T1-GE3, U4 LSM9DS0, U5 SI2366DS-T1-GE3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

Commit message: Finish routing REV1
Just missing increase arm size for motors.
Parts:
- removed JP1: Debugger, SparkFun-Connectors:M04PTH
- removed R4, R7, R8, R9: 100, resistor:R-US_R0805
- added JP2: FTDI, SparkFun-Connectors:FTDI_BASICPTH
- C25, C26, C4: device SparkFun-Capacitors:CAP0805 -> rcl:C-USC0805
- D1, D2, D3, D4: value BAT60J -> BAS16WS; device diode:BAT60J -> Controller:BAS16WS
- J1: device SparkFun-Connectors:AVR_SPI_PRG_6NS -> Controller:AVR_SPI_PRG_6NS
- R10, R3: device SparkFun-Passives:RESISTOR0805-RES -> resistor:R-US_R0805
- S2: value (none) -> SW; device SparkFun-Electromechanical:SWITCH-SPDTPTH -> Controller:SWITCH-SPDTPTH
- U1: device SparkFun-DigitalIC:ATMEGA128RFA1 -> Controller:ATMEGA128RFA1
- U3, U5, U6, U7: value SI2366DS-T1-GE3 -> SI2302CDS-T1-E3; device Vishay_By_element14_Batch_1:SI2366DS-T1-GE3 -> Controller:SI2302CDS-T1-E3
- U4: device IMU_parts:LSM9DS0 -> Controller:LSM9DS0
Connections:
- removed net N$12: R14.1, R9.1, U7.G
- removed net N$14: C7.2, D1.A
- removed net N$19: C13.2, D3.A
- removed net N$27: C14.2, D4.A
- removed net N$5: R11.1, R4.1, U5.G
- removed net N$6: R12.1, R7.1, U3.G
- removed net N$9: R13.1, R8.1, U6.G
- net 3.3V: now also JP2.4; no longer JP1.3
- net GND: now also JP2.6; no longer JP1.4
- net N$29: now also C7.2, D1.A
- net N$31: now also C13.2, D3.A
- net N$32: now also C14.2, D4.A
- net PB4: now also R13.1, U6.G; no longer R8.2
- net PB5: now also R12.1, U3.G; no longer R7.2
- net PE3: now also R14.1, U7.G; no longer R9.2
- net PE4: now also R11.1, U5.G; no longer R4.2
- net RX1: now also JP2.3; no longer JP1.2
- net TX1: now also JP2.2; no longer JP1.1
Other:
- note added: "- Change Package info in Schematic for motor mosfets and diodes. -Change Boom to 805 components -Increase pcb motor arms."
- note removed: "- Change Package info in Schematic for motor mosfets and diodes. -Raplace all 603 pads with 805 pads -Change Boom to 805 components -Shrink GND pad of Microcontroller -Increase pcb motor arms. - Change pads of micro and IMU to longer pads. - Change Serial to Match FTDI ports."
- moved on the sheet: C13, C14, C26, C7, C8, K1, K2, K3, K4, R11, R12, R13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
