File: Master/Jorge/REV1/UCSD_QuadCopter_Rev1.sch (EAGLE design)
At the start: 58 parts, among them J1 ISP, K1 653002114822, K2 653002114822, K3 653002114822, K4 653002114822, U1 ATMEGA128RFA1, U2 TPS73633-DBVT, U3 SI2302CDS-T1-E3, U4 LSM9DS0, U5 SI2302CDS-T1-E3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

Commit message: Latest Multiwii Code & Schematic
Uploading latest code & Schematic (Jorge).
+ Correct IMU ACC & GYRO ORENTATIOn.
+ Adding some parameters to EEPROM by default..
+ Correct Motors Pin Output for (Rear_L, Rear_R, Front_L, Front_R)
Parts:
- C10: value 1uF -> 200uF
- C23: value 1uF -> 100uF
Other:
- note removed: "- Change Package info in Schematic for motor mosfets and diodes. -Change Boom to 805 components -Increase pcb motor arms."
Changed lines of the file:
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@@
 <part name="SUPPLY8" library="supply2" deviceset="GND" device=""/>
 <part name="U2" library="Power" deviceset="TPS73633-DBVT" device=""/>
-<part name="C10" library="resistor" deviceset="C-US" device="C0805" value="1uF"/>
+<part name="C10" library="resistor" deviceset="C-US" device="C0805" value="200uF"/>
 <part name="SUPPLY2" library="supply2" deviceset="GND" device=""/>
 <part name="C12" library="resistor" deviceset="C-US" device="C0805" value="10nF"/>
-<part name="C23" library="resistor" deviceset="C-US" device="C0805" value="1uF"/>
+<part name="C23" library="resistor" deviceset="C-US" device="C0805" value="100uF"/>
 <part name="SUPPLY3" library="supply2" deviceset="GND" device=""/>
 <part name="R2" library="resistor" deviceset="R-US_" device="R0805" value="330"/>
@@
 </text>
 <text x="45.974" y="135.128" size="3.81" layer="97">TODO</text>
-<text x="43.434" y="105.918" size="2.54" layer="97">- Change Package info in Schematic
-for motor mosfets and diodes.
--Change Boom to 805 components
--Increase pcb motor arms.
+<text x="43.434" y="105.918" size="2.54" layer="97">
 </text>
 </plain>
