File: Controller/Eagle/Projects/Controller_acrylic/controller.brd (EAGLE design)
At the start: 280.8 x 115 mm, 5 parts

Commit message: Moved gimbals up for comfort Made connection board
Parts:
- added J1, J2, J3, J4: GIMBAL_3PIN, Controller:JST-3-PTH
- added JP1: (no value), SparkFun-Connectors:1X02_LOCK
- added JP6: (no value), SparkFun-Connectors:1X04
- added R1, R2, R3, R4: (no value), SparkFun-Resistors:1/6W-RES
- moved U$1 15.0 mm to (29.0, 72.5)
- moved U$2 15.0 mm to (221.0, 72.5)
Connections:
- new net 3.3V: JP1.2, R1.2, R2.2, R3.2, R4.2
- new net GND: J1.3, J2.3, J3.3, J4.3, JP1.1
- new net N$1: J4.1, R1.1
- new net N$2: J3.1, R2.1
- new net N$3: J2.1, R3.1
- new net N$4: J1.1, R4.1
- new net N$5: J1.2, JP6.1
- new net N$6: J2.2, JP6.2
- new net N$7: J3.2, JP6.3
- new net N$8: J4.2, JP6.4
Changed lines of the file:
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@@
 <grid distance="1" unitdist="mm" unit="mm" style="lines" multiple="1" display="yes" altdistance="0.001" altunitdist="mm" altunit="mm"/>
 <layers>
-<layer number="1" name="Top" color="4" fill="1" visible="no" active="yes"/>
+<layer number="1" name="Top" color="4" fill="1" visible="yes" active="yes"/>
 <layer number="2" name="Route2" color="1" fill="3" visible="no" active="no"/>
 <layer number="3" name="Route3" color="4" fill="3" visible="no" active="no"/>
@@
 <layer number="14" name="Route14" color="1" fill="6" visible="no" active="no"/>
 <layer number="15" name="Route15" color="4" fill="6" visible="no" active="no"/>
-<layer number="16" name="Bottom" color="1" fill="1" visible="no" active="yes"/>
-<layer number="17" name="Pads" color="2" fill="1" visible="no" active="yes"/>
-<layer number="18" name="Vias" color="2" fill="1" visible="no" active="yes"/>
-<layer number="19" name="Unrouted" color="6" fill="1" visible="no" active="yes"/>
+<layer number="16" name="Bottom" color="1" fill="1" visible="yes" active="yes"/>
+<layer number="17" name="Pads" color="2" fill="1" visible="yes" active="yes"/>
+<layer number="18" name="Vias" color="2" fill="1" visible="yes" active="yes"/>
+<layer number="19" name="Unrouted" color="6" fill="1" visible="yes" active="yes"/>
 <layer number="20" name="Dimension" color="15" fill="1" visible="yes" active="yes"/>
-<layer number="21" name="tPlace" color="7" fill="1" visible="no" active="yes"/>
-<layer number="22" name="bPlace" color="7" fill="1" visible="no" active="yes"/>
-<layer number="23" name="tOrigins" color="15" fill="1" visible="no" active="yes"/>
-<layer number="24" name="bOrigins" color="15" fill="1" visible="no" active="yes"/>
-<layer number="25" name="tNames" color="7" fill="1" visible="no" active="yes"/>
-<layer number="26" name="bNames" color="7" fill="1" visible="no" active="yes"/>
-<layer number="27" name="tValues" color="7" fill="1" visible="no" active="yes"/>
-<layer number="28" name="bValues" color="7" fill="1" visible="no" active="yes"/>
+<layer number="21" name="tPlace" color="7" fill="1" visible="yes" active="yes"/>
+<layer number="22" name="bPlace" color="7" fill="1" visible="yes" active="yes"/>
+<layer number="23" name="tOrigins" color="15" fill="1" visible="yes" active="yes"/>
+<layer number="24" name="bOrigins" color="15" fill="1" visible="yes" active="yes"/>
+<layer number="25" name="tNames" color="7" fill="1" visible="yes" active="yes"/>
+<layer number="26" name="bNames" color="7" fill="1" visible="yes" active="yes"/>
+<layer number="27" name="tValues" color="7" fill="1" visible="yes" active="yes"/>
+<layer number="28" name="bValues" color="7" fill="1" visible="yes" active="yes"/>
 <layer number="29" name="tStop" color="7" fill="3" visible="no" active="yes"/>
 <layer number="30" name="bStop" color="7" fill="6" visible="no" active="yes"/>
@@
 <layer number="39" name="tKeepout" color="4" fill="11" visible="no" active="yes"/>
 <layer number="40" name="bKeepout" color="1" fill="11" visible="no" active="yes"/>
-<layer number="41" name="tRestrict" color="4" fill="10" visible="no" active="yes"/>
+<layer number="41" name="tRestrict" color="4" fill="10" visible="yes" active="yes"/>
 <layer number="42" name="bRestrict" color="1" fill="10" visible="no" active="yes"/>
 <layer number="43" name="vRestrict" color="2" fill="10" visible="no" active="yes"/>
@@
 <layer number="223" name="223bmp" color="7" fill="1" visible="no" active="yes"/>
 <layer number="224" name="224bmp" color="7" fill="1" visible="no" active="yes"/>
+<layer number="225" name="225bmp" color="7" fill="1" visible="yes" active="yes"/>
+<layer number="226" name="226bmp" color="7" fill="1" visible="yes" active="yes"/>
+<layer number="227" name="227bmp" color="7" fill="1" visible="yes" active="yes"/>
+<layer number="228" name="228bmp" color="7" fill="1" visible="yes" active="yes"/>
+<layer number="229" name="229bmp" color="7" fill="1" visible="yes" active="yes"/>
+<layer number="230" name="230bmp" color="7" fill="1" visible="yes" active="yes"/>
+<layer number="231" name="231bmp" color="7" fill="1" visible="yes" active="yes"/>
 <layer number="248" name="Housing" color="7" fill="1" visible="no" active="yes"/>
 <layer number="249" name="Edge" color="7" fill="1" visible="no" active="yes"/>
@@
 </class>
 </classes>
-<designrules name="4pcb-33board">
+<designrules name="4pcb-33board *">
 <description language="de">&lt;b&gt;EAGLE Design Rules&lt;/b&gt;
 &lt;p&gt;
@@
 <param name="mdSmdStop" value="0mil"/>
 <param name="msWidth" value="10mil"/>
-<param name="msDrill" value="15mil"/>
+<param name="msDrill" value="0.9mm"/>
 <param name="msMicroVia" value="9.98981875mm"/>
 <param name="msBlindViaRatio" value="0.5"/>
@@
 <elements>
 <element name="U$3" library="BOBs" package="ATMEGA128RFA1" value="" x="170" y="114" rot="MR270"/>
-<element name="U$1" library="Controller" package="GIMBAL_FOOTPRINT" value="" x="30" y="57.5"/>
-<element name="U$2" library="Controller" package="GIMBAL_FOOTPRINT" value="" x="220" y="57.5"/>
+<element name="U$1" library="Controller" package="GIMBAL_FOOTPRINT" value="" x="29" y="72.5"/>
+<element name="U$2" library="Controller" package="GIMBAL_FOOTPRINT" value="" x="221" y="72.5"/>
 <element name="U$4" library="Controller" package="SPARKFUN_LCD_33" value="" x="83" y="1"/>
 <element name="U$5" library="Controller" package="CONTROLLER_OUTLINE" value="" x="0" y="0"/>
+<element name="J1" library="Controller" package="JST-3-PTH" value="GIMBAL_3PIN" x="189" y="57" rot="R90"/>
+<element name="J2" library="Controller" package="JST-3-PTH" value="GIMBAL_3PIN" x="211" y="39" rot="R180"/>
+<element name="J3" library="Controller" package="JST-3-PTH" value="GIMBAL_3PIN" x="70" y="55" rot="R270"/>
+<element name="J4" library="Controller" package="JST-3-PTH" value="GIMBAL_3PIN" x="43" y="36" rot="R180"/>
+<element name="R1" library="SparkFun-Resistors" package="1/6W-RES" value="" x="62.780953125" y="38.318003125"/>
+<element name="R2" library="SparkFun-Resistors" package="1/6W-RES" value="" x="72.949403125" y="45.939940625"/>
+<element name="R3" library="SparkFun-Resistors" package="1/6W-RES" value="" x="201.042509375" y="42.352325" rot="R270"/>
+<element name="R4" library="SparkFun-Resistors" package="1/6W-RES" value="" x="175.58266875" y="48.739028125" rot="R270"/>
+<element name="JP6" library="SparkFun-Connectors" package="1X04" value="" x="124" y="46" rot="R90"/>
+<element name="JP1" library="SparkFun-Connectors" package="1X02_LOCK" value="" x="113" y="54" rot="R180"/>
 </elements>
 <signals>
+<signal name="GND">
+<contactref element="J4" pad="3"/>
+<contactref element="J1" pad="3"/>
+<contactref element="J2" pad="3"/>
+<contactref element="J3" pad="3"/>
+<contactref element="JP1" pad="1"/>
+<wire x1="209" y1="39" x2="189" y2="59" width="0" layer="19" extent="1-1"/>
+<wire x1="113.1778" y1="54" x2="189" y2="59" width="0" layer="19" extent="1-1"/>
+<wire x1="70" y1="53" x2="113.1778" y2="54" width="0" layer="19" extent="1-1"/>
+<wire x1="41" y1="36" x2="70" y2="53" width="0" layer="19" extent="1-1"/>
+</signal>
+<signal name="N$1">
+<contactref element="J4" pad="1"/>
+<contactref element="R1" pad="1"/>
+<wire x1="45" y1="36" x2="60.280953125" y2="38.318003125" width="0" layer="19" extent="1-1"/>
+</signal>
+<signal name="N$2">
+<contactref element="J3" pad="1"/>
+<contactref element="R2" pad="1"/>
+<wire x1="70.449403125" y1="45.939940625" x2="70" y2="57" width="0" layer="19" extent="1-1"/>
+</signal>
+<signal name="N$3">
+<contactref element="J2" pad="1"/>
+<contactref element="R3" pad="1"/>
+<wire x1="201.042509375" y1="44.852325" x2="213" y2="39" width="0" layer="19" extent="1-1"/>
+</signal>
+<signal name="N$4">
+<contactref element="J1" pad="1"/>
+<contactref element="R4" pad="1"/>
+<wire x1="175.58266875" y1="51.239028125" x2="189" y2="55" width="0" layer="19" extent="1-1"/>
+</signal>
+<signal name="3.3V">
+<contactref element="R4" pad="2"/>
+<contactref element="R3" pad="2"/>
+<contactref element="R2" pad="2"/>
+<contactref element="R1" pad="2"/>
+<contactref element="JP1" pad="2"/>
+<wire x1="175.58266875" y1="46.239028125" x2="201.042509375" y2="39.852325" width="0" layer="19" extent="1-1"/>
+<wire x1="110.2822" y1="54" x2="175.58266875" y2="46.239028125" width="0" layer="19" extent="1-1"/>
+<wire x1="75.449403125" y1="45.939940625" x2="110.2822" y2="54" width="0" layer="19" extent="1-1"/>
+<wire x1="65.280953125" y1="38.318003125" x2="75.449403125" y2="45.939940625" width="0" layer="19" extent="1-1"/>
+</signal>
+<signal name="N$5">
+<contactref element="J1" pad="2"/>
+<contactref element="JP6" pad="1"/>
+<wire x1="124" y1="46" x2="189" y2="57" width="0" layer="19" extent="1-1"/>
+</signal>
+<signal name="N$6">
+<contactref element="J2" pad="2"/>
+<contactref element="JP6" pad="2"/>
+<wire x1="124" y1="48.54" x2="211" y2="39" width="0" layer="19" extent="1-1"/>
+</signal>
+<signal name="N$7">
+<contactref element="J3" pad="2"/>
+<contactref element="JP6" pad="3"/>
+<wire x1="70" y1="55" x2="124" y2="51.08" width="0" layer="19" extent="1-1"/>
+</signal>
+<signal name="N$8">
+<contactref element="J4" pad="2"/>
+<contactref element="JP6" pad="4"/>
+<wire x1="43" y1="36" x2="124" y2="53.62" width="0" layer="19" extent="1-1"/>
+</signal>
 </signals>
 </board>
