File: Controller/Eagle/Projects/Controller_acrylic/controller.sch (EAGLE design)
At the start: 0 parts

Commit message: Moved gimbals up for comfort Made connection board
Parts:
- added J1, J2, J3, J4: GIMBAL_3PIN, Controller:GIMBAL_3PIN
- added JP1: (no value), SparkFun-Connectors:M02LOCK
- added JP6: (no value), SparkFun-Connectors:M04PTH
- added R1, R2, R3, R4: (no value), SparkFun-Resistors:RESISTORPTH-1/6W
Connections:
- new net 3.3V: JP1.2, R1.2, R2.2, R3.2, R4.2
- new net GND: J1.GND, J2.GND, J3.GND, J4.GND, JP1.1
- new net N$1: J4.VDD, R1.1
- new net N$2: J3.VDD, R2.1
- new net N$3: J2.VDD, R3.1
- new net N$4: J1.VDD, R4.1
- new net N$5: J1.AOUT, JP6.1
- new net N$6: J2.AOUT, JP6.2
- new net N$7: J3.AOUT, JP6.3
- new net N$8: J4.AOUT, JP6.4
Changed lines of the file:
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@@
 <setting verticaltext="up"/>
 </settings>
-<grid distance="0.1" unitdist="inch" unit="inch" style="lines" multiple="1" display="yes" altdistance="0.01" altunitdist="inch" altunit="inch"/>
+<grid distance="0.1" unitdist="inch" unit="inch" style="lines" multiple="1" display="no" altdistance="0.01" altunitdist="inch" altunit="inch"/>
 <layers>
 <layer number="1" name="Top" color="4" fill="1" visible="no" active="no"/>
@@
 <layer number="154" name="FabDoc2" color="7" fill="1" visible="yes" active="yes"/>
 <layer number="155" name="FabDoc3" color="7" fill="1" visible="yes" active="yes"/>
+<layer number="160" name="tMountFaceplate" color="11" fill="1" visible="no" active="yes"/>
+<layer number="161" name="bMountFaceplate" color="11" fill="1" visible="no" active="yes"/>
 <layer number="199" name="Contour" color="7" fill="1" visible="yes" active="yes"/>
 <layer number="200" name="200bmp" color="7" fill="1" visible="yes" active="yes"/>
@@
 <layer number="223" name="223bmp" color="7" fill="1" visible="yes" active="yes"/>
 <layer number="224" name="224bmp" color="7" fill="1" visible="yes" active="yes"/>
+<layer number="225" name="225bmp" color="7" fill="1" visible="yes" active="yes"/>
+<layer number="226" name="226bmp" color="7" fill="1" visible="yes" active="yes"/>
+<layer number="227" name="227bmp" color="7" fill="1" visible="yes" active="yes"/>
+<layer number="228" name="228bmp" color="7" fill="1" visible="yes" active="yes"/>
+<layer number="229" name="229bmp" color="7" fill="1" visible="yes" active="yes"/>
+<layer number="230" name="230bmp" color="7" fill="1" visible="yes" active="yes"/>
+<layer number="231" name="231bmp" color="7" fill="1" visible="yes" active="yes"/>
 <layer number="248" name="Housing" color="7" fill="1" visible="yes" active="yes"/>
 <layer number="249" name="Edge" color="7" fill="1" visible="yes" active="yes"/>
@@
 </classes>
 <parts>
+<part name="J1" library="Controller" deviceset="GIMBAL_3PIN" device=""/>
+<part name="J2" library="Controller" deviceset="GIMBAL_3PIN" device=""/>
+<part name="J3" library="Controller" deviceset="GIMBAL_3PIN" device=""/>
+<part name="J4" library="Controller" deviceset="GIMBAL_3PIN" device=""/>
+<part name="R1" library="SparkFun-Resistors" deviceset="RESISTOR" device="PTH-1/6W"/>
+<part name="R2" library="SparkFun-Resistors" deviceset="RESISTOR" device="PTH-1/6W"/>
+<part name="R3" library="SparkFun-Resistors" deviceset="RESISTOR" device="PTH-1/6W"/>
+<part name="R4" library="SparkFun-Resistors" deviceset="RESISTOR" device="PTH-1/6W"/>
+<part name="JP6" library="SparkFun-Connectors" deviceset="M04" device="PTH"/>
+<part name="JP1" library="SparkFun-Connectors" deviceset="M02" device="LOCK"/>
 </parts>
 <sheets>
@@
 </plain>
 <instances>
+<instance part="J1" gate="G$1" x="33.02" y="71.12" rot="R180"/>
+<instance part="J2" gate="G$1" x="33.02" y="53.34" rot="R180"/>
+<instance part="J3" gate="G$1" x="33.02" y="33.02" rot="R180"/>
+<instance part="J4" gate="G$1" x="33.02" y="17.78" rot="R180"/>
+<instance part="R1" gate="G$1" x="55.88" y="10.16"/>
+<instance part="R2" gate="G$1" x="55.88" y="25.4"/>
+<instance part="R3" gate="G$1" x="55.88" y="45.72"/>
+<instance part="R4" gate="G$1" x="55.88" y="63.5"/>
+<instance part="JP6" gate="G$1" x="104.14" y="43.18" rot="R180"/>
+<instance part="JP1" gate="G$1" x="68.58" y="78.74" rot="R180"/>
 </instances>
 <busses>
 </busses>
 <nets>
+<net name="GND" class="0">
+<segment>
+<pinref part="J4" gate="G$1" pin="GND"/>
+<wire x1="38.1" y1="15.24" x2="43.18" y2="15.24" width="0.1524" layer="91"/>
+<wire x1="43.18" y1="15.24" x2="43.18" y2="30.48" width="0.1524" layer="91"/>
+<pinref part="J1" gate="G$1" pin="GND"/>
+<wire x1="43.18" y1="30.48" x2="43.18" y2="50.8" width="0.1524" layer="91"/>
+<wire x1="43.18" y1="50.8" x2="43.18" y2="68.58" width="0.1524" layer="91"/>
+<wire x1="43.18" y1="68.58" x2="38.1" y2="68.58" width="0.1524" layer="91"/>
+<pinref part="J2" gate="G$1" pin="GND"/>
+<wire x1="38.1" y1="50.8" x2="43.18" y2="50.8" width="0.1524" layer="91"/>
+<pinref part="J3" gate="G$1" pin="GND"/>
+<wire x1="38.1" y1="30.48" x2="43.18" y2="30.48" width="0.1524" layer="91"/>
+<junction x="43.18" y="30.48"/>
+<junction x="43.18" y="50.8"/>
+<wire x1="43.18" y1="68.58" x2="43.18" y2="78.74" width="0.1524" layer="91"/>
+<pinref part="JP1" gate="G$1" pin="1"/>
+<wire x1="43.18" y1="78.74" x2="60.96" y2="78.74" width="0.1524" layer="91"/>
+<junction x="43.18" y="68.58"/>
+</segment>
+</net>
+<net name="N$1" class="0">
+<segment>
+<pinref part="J4" gate="G$1" pin="VDD"/>
+<pinref part="R1" gate="G$1" pin="1"/>
+<wire x1="38.1" y1="10.16" x2="50.8" y2="10.16" width="0.1524" layer="91"/>
+</segment>
+</net>
+<net name="N$2" class="0">
+<segment>
+<pinref part="J3" gate="G$1" pin="VDD"/>
+<pinref part="R2" gate="G$1" pin="1"/>
+<wire x1="38.1" y1="25.4" x2="50.8" y2="25.4" width="0.1524" layer="91"/>
+</segment>
+</net>
+<net name="N$3" class="0">
+<segment>
+<pinref part="J2" gate="G$1" pin="VDD"/>
+<pinref part="R3" gate="G$1" pin="1"/>
+<wire x1="38.1" y1="45.72" x2="50.8" y2="45.72" width="0.1524" layer="91"/>
+</segment>
+</net>
+<net name="N$4" class="0">
+<segment>
+<pinref part="J1" gate="G$1" pin="VDD"/>
+<pinref part="R4" gate="G$1" pin="1"/>
+<wire x1="38.1" y1="63.5" x2="50.8" y2="63.5" width="0.1524" layer="91"/>
+</segment>
+</net>
+<net name="3.3V" class="0">
+<segment>
+<pinref part="R4" gate="G$1" pin="2"/>
+<pinref part="R3" gate="G$1" pin="2"/>
+<wire x1="60.96" y1="63.5" x2="60.96" y2="45.72" width="0.1524" layer="91"/>
+<pinref part="R2" gate="G$1" pin="2"/>
+<wire x1="60.96" y1="45.72" x2="60.96" y2="25.4" width="0.1524" layer="91"/>
+<pinref part="R1" gate="G$1" pin="2"/>
+<wire x1="60.96" y1="25.4" x2="60.96" y2="10.16" width="0.1524" layer="91"/>
+<junction x="60.96" y="45.72"/>
+<junction x="60.96" y="25.4"/>
+<junction x="60.96" y="10.16"/>
+<junction x="60.96" y="63.5"/>
+<pinref part="JP1" gate="G$1" pin="2"/>
+<wire x1="60.96" y1="76.2" x2="60.96" y2="63.5" width="0.1524" layer="91"/>
+</segment>
+</net>
+<net name="N$5" class="0">
+<segment>
+<pinref part="J1" gate="G$1" pin="AOUT"/>
+<wire x1="38.1" y1="66.04" x2="99.06" y2="66.04" width="0.1524" layer="91"/>
+<pinref part="JP6" gate="G$1" pin="1"/>
+<wire x1="99.06" y1="66.04" x2="99.06" y2="45.72" width="0.1524" layer="91"/>
+</segment>
+</net>
+<net name="N$6" class="0">
+<segment>
+<pinref part="J2" gate="G$1" pin="AOUT"/>
+<wire x1="86.36" y1="48.26" x2="38.1" y2="48.26" width="0.1524" layer="91"/>
+<wire x1="86.36" y1="48.26" x2="86.36" y2="43.18" width="0.1524" layer="91"/>
+<pinref part="JP6" gate="G$1" pin="2"/>
+<wire x1="86.36" y1="43.18" x2="99.06" y2="43.18" width="0.1524" layer="91"/>
+</segment>
+</net>
+<net name="N$7" class="0">
+<segment>
+<pinref part="J3" gate="G$1" pin="AOUT"/>
+<wire x1="38.1" y1="27.94" x2="86.36" y2="27.94" width="0.1524" layer="91"/>
+<wire x1="86.36" y1="27.94" x2="86.36" y2="40.64" width="0.1524" layer="91"/>
+<pinref part="JP6" gate="G$1" pin="3"/>
+<wire x1="86.36" y1="40.64" x2="99.06" y2="40.64" width="0.1524" layer="91"/>
+</segment>
+</net>
+<net name="N$8" class="0">
+<segment>
+<pinref part="J4" gate="G$1" pin="AOUT"/>
+<wire x1="93.98" y1="12.7" x2="38.1" y2="12.7" width="0.1524" layer="91"/>
+<wire x1="93.98" y1="12.7" x2="93.98" y2="38.1" width="0.1524" layer="91"/>
+<pinref part="JP6" gate="G$1" pin="4"/>
+<wire x1="93.98" y1="38.1" x2="99.06" y2="38.1" width="0.1524" layer="91"/>
+</segment>
+</net>
 </nets>
 </sheet>
