File: Controller/Eagle/Projects/Controller_acrylic/controller_top.brd (EAGLE design)
At the start: 280.8 x 115 mm, 2 parts

Commit message: Organized eagle files better
Top: top faceplate
Bottom: bottom faceplate (both acrylic)
connector_board: PCB to connect stuff to
Parts:
- added U$1, U$2: (no value), Controller:GIMBAL_FOOTPRINT
- added U$4: (no value), Controller:SPARKFUN_LCD_33
- moved U$3 44.0 mm to (170.0, 114.0), flipped to the bottom
Changed lines of the file:
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@@
 <setting verticaltext="up"/>
 </settings>
-<grid distance="1" unitdist="mm" unit="mm" style="lines" multiple="1" display="yes" altdistance="0.5" altunitdist="mm" altunit="mm"/>
+<grid distance="1" unitdist="mm" unit="mm" style="lines" multiple="1" display="yes" altdistance="0.001" altunitdist="mm" altunit="mm"/>
 <layers>
 <layer number="1" name="Top" color="4" fill="1" visible="no" active="yes"/>
@@
 <layer number="223" name="223bmp" color="7" fill="1" visible="no" active="yes"/>
 <layer number="224" name="224bmp" color="7" fill="1" visible="no" active="yes"/>
+<layer number="225" name="225bmp" color="7" fill="1" visible="no" active="yes"/>
+<layer number="226" name="226bmp" color="7" fill="1" visible="no" active="yes"/>
+<layer number="227" name="227bmp" color="7" fill="1" visible="no" active="yes"/>
+<layer number="228" name="228bmp" color="7" fill="1" visible="no" active="yes"/>
+<layer number="229" name="229bmp" color="7" fill="1" visible="no" active="yes"/>
+<layer number="230" name="230bmp" color="7" fill="1" visible="no" active="yes"/>
+<layer number="231" name="231bmp" color="7" fill="1" visible="no" active="yes"/>
+<layer number="232" name="Eagle3D_PG2" color="7" fill="1" visible="no" active="no"/>
+<layer number="233" name="Eagle3D_PG3" color="7" fill="1" visible="no" active="no"/>
 <layer number="248" name="Housing" color="7" fill="1" visible="no" active="yes"/>
 <layer number="249" name="Edge" color="7" fill="1" visible="no" active="yes"/>
@@
 </class>
 </classes>
-<designrules name="4pcb-33board">
+<designrules name="4pcb-33board *">
 <description language="de">&lt;b&gt;EAGLE Design Rules&lt;/b&gt;
 &lt;p&gt;
@@
 <param name="mdSmdStop" value="0mil"/>
 <param name="msWidth" value="10mil"/>
-<param name="msDrill" value="15mil"/>
+<param name="msDrill" value="0.9mm"/>
 <param name="msMicroVia" value="9.98981875mm"/>
 <param name="msBlindViaRatio" value="0.5"/>
@@
 </autorouter>
 <elements>
-<element name="U$3" library="BOBs" package="ATMEGA128RFA1" value="" x="126" y="114" rot="R270"/>
+<element name="U$3" library="BOBs" package="ATMEGA128RFA1" value="" x="170" y="114" rot="MR270"/>
+<element name="U$1" library="Controller" package="GIMBAL_FOOTPRINT" value="" x="29" y="72.5"/>
+<element name="U$2" library="Controller" package="GIMBAL_FOOTPRINT" value="" x="221" y="72.5"/>
+<element name="U$4" library="Controller" package="SPARKFUN_LCD_33" value="" x="82.938" y="2.814"/>
 <element name="U$5" library="Controller" package="CONTROLLER_OUTLINE" value="" x="0" y="0"/>
 </elements>

Commit message: Moved both gimbals 5mm closer to the edge for comfort
Parts:
- moved U$1 5.00 mm to (24.0, 72.5)
- moved U$2 5.00 mm to (226.0, 72.5)
Changed lines of the file:
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@@
 <elements>
 <element name="U$3" library="BOBs" package="ATMEGA128RFA1" value="" x="170" y="114" rot="MR270"/>
-<element name="U$1" library="Controller" package="GIMBAL_FOOTPRINT" value="" x="29" y="72.5"/>
-<element name="U$2" library="Controller" package="GIMBAL_FOOTPRINT" value="" x="221" y="72.5"/>
+<element name="U$1" library="Controller" package="GIMBAL_FOOTPRINT" value="" x="24" y="72.5"/>
+<element name="U$2" library="Controller" package="GIMBAL_FOOTPRINT" value="" x="226" y="72.5"/>
 <element name="U$4" library="Controller" package="SPARKFUN_LCD_33" value="" x="82.938" y="2.814"/>
 <element name="U$5" library="Controller" package="CONTROLLER_OUTLINE" value="" x="0" y="0"/>
